Commit message: for the demo- camera and laser on power base

File: mrs_description/robots/power_base.xacro (robot description, xacro)
@@ -3,7 +3,7 @@
   <!-- The following included files set up definitions of parts of the robot body -->
   <!-- power base -->
-  <include filename="$(find mrs_description)/urdf/power_base/base.urdf.xacro" />
+  <xacro:include filename="$(find mrs_description)/urdf/power_base/base.urdf.xacro" />
   <!-- materials for visualization -->
-  <include filename="$(find mrs_description)/urdf/materials.urdf.xacro" />
+  <xacro:include filename="$(find mrs_description)/urdf/materials.urdf.xacro" />
   <!-- Now we can start using the macros included above to define the actual power -->
   <!-- The first use of a macro.  This one was defined in base.urdf.xacro above.
@@ -20,4 +20,5 @@
   <xacro:Ball_bearing mass="0.1" instance="3" dia="0.05" x="0.05" y="-0.05" z="-0.05" parent="base_link"/>
   <xacro:Ball_bearing mass="0.1" instance="4" dia="0.05" x="-0.05" y="-0.05" z="-0.05" parent="base_link"/>
+<!--
   <gazebo>
     <plugin name="gazebo_ros_controller_manager" filename="libgazebo_ros_control.so">
@@ -32,3 +33,4 @@
     </plugin>
   </gazebo>
+-->
 </robot>

File: mrs_description/urdf/power_base/base.urdf.xacro (robot description, xacro)
@@ -2,84 +2,96 @@
 <robot xmlns:xacro="http://www.ros.org/wiki/xacro">
 <xacro:include filename="$(find mrs_description)/urdf/power_base/ball_bearing.urdf.xacro" />
-		<!-- Constants for robot -->
-	<xacro:include filename="$(find mrs_description)/urdf/common_mrs.xacro" />
+		<!-- constants for robot -->
+<xacro:include filename="$(find mrs_description)/urdf/common_mrs.xacro" />
   <!-- simplified box collision geometry for base -->
+<xacro:include filename="$(find
+mrs_description)/urdf/power_base/sm_other.urdf.xacro" />
   <property name="mass" value="22.0"/>
-  	<property name="P_baselen" value=".3" />
-	<property name="P_basewidth" value=".3" />
-	<property name="P_baseheight" value=".1" />
+  <property name="p_baselen" value=".3" />
+	<property name="p_basewidth" value=".3" />
+	<property name="p_baseheight" value=".1" />
   <xacro:macro name="power_base" params="name">
-    <link name="${name}_footprint">
-      <inertial>
-        <mass value="0.1"/>
-        <origin xyz="0 0 ${-P_baseheight/2}" rpy="0 0 0"/>
-        <inertia ixx="1.0" ixy="0.0" ixz="0.0" iyy="1.0" iyz="0.0" izz="1.0"/>
-      </inertial>
-      <visual>
-        <origin xyz="0 0 0" rpy="0 0 0"/>
-        <geometry>
-          <box size="0.001 0.001 0.001"/>
-        </geometry>
-        <material name="Red"/>
-      </visual>
-      <collision>
-        <origin xyz="0 0 ${-P_baseheight/2}" rpy="0 0 0"/>
-        <geometry>
-          <box size="0.001 0.001 0.001"/>
-        </geometry>
-      </collision>
-    </link>
-    <joint name="${name}_footprint_joint" type="fixed">
+  <link name="${name}_footprint">
+    <inertial>
+      <mass value="0.1"/>
+      <origin xyz="0 0 ${-p_baseheight/2}" rpy="0 0 0"/>
+      <inertia ixx="1.0" ixy="0.0" ixz="0.0" iyy="1.0" iyz="0.0" izz="1.0"/>
+    </inertial>
+    <visual>
       <origin xyz="0 0 0" rpy="0 0 0"/>
-      <child link="${name}_link"/>
-      <parent link="${name}_footprint"/>
-    </joint>
-    <link name="${name}_link">
-      <inertial>
-        <mass value="${mass}"/>
-        <inertia ixx="${1/12*mass*(P_baselen*P_baselen+P_baseheight*P_baseheight)}" ixy="0" ixz="0" iyy="${1/12*mass*(P_basewidth*P_basewidth+P_baselen*P_baselen)}" iyz="0" izz="${1/12*mass*(P_basewidth*P_basewidth+P_baseheight*P_baseheight)}"/>
-        <origin xyz="0 0 0"/>
-      </inertial>
-		<visual>
-			<geometry>
-				<cylinder radius="${P_basewidth+0.05}" length="${P_baseheight}" />
-			</geometry>
-			<material name="Green">
-			</material>
-		</visual>
-		<collision>
-			<geometry>
-				<cylinder radius="${P_basewidth}" length="${P_baseheight}" />
-			</geometry>
-		</collision>
-    </link>
-			<gazebo reference="${name}_link">
-     			<material>Gazebo/Grey</material>
-    		</gazebo>
-	<joint name="${name}_link_support_joint" type="fixed">
-		<origin xyz="0 0 ${P_baseheight*6/2}" rpy="0 0 0" />
-		<child link="${name}_link_support" />
-		<parent link="${name}_link" />
-	</joint>
-	<link name="${name}_link_support">
-		      <visual>
-        <geometry>
-          <box size="${P_baselen} ${P_basewidth} ${P_baseheight*6}" />
-        </geometry>
-        <material name="DarkGrey"/>
-      </visual>
-      <collision>
-        <geometry>
-          <box size="${P_baselen-0.1} ${P_basewidth-0.05} ${P_baseheight*6-0.05}" />
-        </geometry>
-      </collision>
-		<xacro:default_inertial mass="2" />
-	</link>
-			<gazebo reference="${name}_link_support">
-     			<material>Gazebo/Grey</material>
-    		</gazebo>
+      <geometry>
+        <box size="0.001 0.001 0.001"/>
+      </geometry>
+      <material name="red"/>
+    </visual>
+    <collision>
+      <origin xyz="0 0 ${-p_baseheight/2}" rpy="0 0 0"/>
+      <geometry>
+        <box size="0.001 0.001 0.001"/>
+      </geometry>
+    </collision>
+  </link>
+  <joint name="${name}_footprint_joint" type="fixed">
+    <origin xyz="0 0 0" rpy="0 0 0"/>
+    <child link="${name}_link"/>
+    <parent link="${name}_footprint"/>
+  </joint>
+  <link name="${name}_link">
+  <inertial>
+    <mass value="${mass}"/>
+    <inertia ixx="${1/12*mass*(p_baselen*p_baselen+p_baseheight*p_baseheight)}" ixy="0" ixz="0" iyy="${1/12*mass*(p_basewidth*p_basewidth+p_baselen*p_baselen)}" iyz="0" izz="${1/12*mass*(p_basewidth*p_basewidth+p_baseheight*p_baseheight)}"/>
+    <origin xyz="0 0 0"/>
+  </inertial>
+  <visual>
+    <geometry>
+      <cylinder radius="${p_basewidth+0.05}" length="${p_baseheight}" />
+    </geometry>
+    <material name="White">
+    </material>
+  </visual>
+  <collision>
+    <geometry>
+      <cylinder radius="${p_basewidth}" length="${p_baseheight}" />
+    </geometry>
+  </collision>
+  </link>
+  <gazebo reference="${name}_link">
+    <material>Gazebo/Grey</material>
+  </gazebo>
+  <joint name="${name}_link_support_joint" type="fixed">
+    <origin xyz="0 0 ${p_baseheight*6/2}" rpy="0 0 0" />
+    <child link="${name}_link_support" />
+    <parent link="${name}_link" />
+  </joint>
+  <link name="${name}_link_support">
+    <visual>
+      <geometry>
+        <box size="${p_baselen} ${p_basewidth} ${p_baseheight*6}" />
+      </geometry>
+      <material name="Orange"/>
+    </visual>
+    <collision>
+      <geometry>
+        <box size="${p_baselen-0.1} ${p_basewidth-0.05} ${p_baseheight*6-0.05}" />
+      </geometry>
+    </collision>
+    <xacro:default_inertial mass="2" />
+  </link>
+  <gazebo reference="${name}_link_support">
+    <material>Gazebo/Grey</material>
+  </gazebo>
   </xacro:macro>
+<xacro:Camera parent="base_link_support" prefix="base" x="0.15"
+y="0" z="0.27" instance="1" />
+<xacro:Camera parent="base_link_support" prefix="base" x="0"
+y="0.15" z="0.27" instance="2" />
+<xacro:Camera parent="base_link_support" prefix="base" x="-0.15"
+y="0" z="0.27" instance="3" />
+<xacro:Camera parent="base_link_support" prefix="base" x="0"
+y="-0.15" z="0.27" instance="4" />
+<xacro:Laser parent="base_link_support" prefix="base" x="0"
+y="0" z="0.31" instance="1" />
 <!--
-   <xacro:Ball_bearing mass="0.1" instance="1" dia="0.05" x="0" y="0" z="-0.05" parent="base_link"/>
+   <xacro:ball_bearing mass="0.1" instance="1" dia="0.05" x="0" y="0" z="-0.05" parent="base_link"/>
 -->
 </robot>

File: mrs_description/urdf/power_base/sm_other.urdf.xacro (robot description, xacro)
@@ -5,4 +5,122 @@
   <!-- simplified box collision geometry for base -->
   <property name="mass" value="22.0"/>
+   <!-- Size of square 'camera' box -->
+  <xacro:property name="camera_size" value="0.05" />
+	<xacro:macro name="Camera" params="parent prefix x y z instance">
+    <joint name="${instance}_${prefix}_camera_joint" type="fixed">
+      <axis xyz="1 0 0" />
+      <parent link="${parent}" />
+      <child link="${instance}_${prefix}_camera_link" />
+      <origin rpy="0 0 0" xyz="${x} ${y} ${z}" />
+    </joint>
+    <link name="${instance}_${prefix}_camera_link">
+      <visual>
+        <geometry>
+          	<box size="${camera_size} ${camera_size} ${camera_size}"/>
+        </geometry>
+        <origin rpy="0 0 0 " xyz="0 0 0" />
+        <material name="Red"/>
+      </visual>
+      <collision>
+        <origin rpy="0 0 0 " xyz="0 0 0" />
+        <geometry>
+          	<box size="${camera_size} ${camera_size} ${camera_size}"/>
+        </geometry>
+      </collision>
+      <inertial>
+        <mass value="1e-5" />
+        <origin xyz="0 0 0" rpy="0 0 0"/>
+        <inertia ixx="1e-6" ixy="0" ixz="0" iyy="1e-6" iyz="0" izz="1e-6" />
+      </inertial>
+    </link>
+    <gazebo reference="${instance}_${prefix}_camera_link">
+      <mu1>0.2</mu1>
+      <mu2>0.2</mu2>
+      <material>Gazebo/Red</material>
+      <sensor type="camera" name="${instance}_${prefix}_camera">
+      <update_rate>30.0</update_rate>
+        <camera name="${instance}_${prefix}_camera">
+          <horizontal_fov>1.3962634</horizontal_fov>
+          <image>
+            <width>800</width>
+            <height>800</height>
+            <format>R8G8B8</format>
+          </image>
+          <clip>
+            <near>0.02</near>
+            <far>300</far>
+          </clip>
+        </camera>
+        <plugin name="camera_controller" filename="libgazebo_ros_camera.so">
+          <alwaysOn>true</alwaysOn>
+          <updateRate>0.0</updateRate>
+          <cameraName>mrs/${instance}_${prefix}_camera</cameraName>
+          <imageTopicName>image_raw</imageTopicName>
+          <cameraInfoTopicName>camera_info</cameraInfoTopicName>
+          <frameName>camera_link</frameName>
+          <hackBaseline>0.07</hackBaseline>
+          <distortionK1>0.0</distortionK1>
+          <distortionK2>0.0</distortionK2>
+          <distortionK3>0.0</distortionK3>
+          <distortionT1>0.0</distortionT1>
+          <distortionT2>0.0</distortionT2>
+        </plugin>
+      </sensor>
+    </gazebo>
+	</xacro:macro>
+	<xacro:macro name="Laser" params="parent prefix x y z instance">
+    <joint name="${instance}_${prefix}_laser_joint" type="fixed">
+      <axis xyz="1 0 0" />
+      <parent link="${parent}" />
+      <child link="${instance}_${prefix}_laser_link" />
+      <origin rpy="0 0 0" xyz="${x} ${y} ${z}" />
+    </joint>
+    <link name="${instance}_${prefix}_laser_link">
+      <visual>
+        <geometry>
+          	<box size="${camera_size} ${camera_size} ${camera_size}"/>
+        </geometry>
+        <origin rpy="0 0 0 " xyz="0 0 0" />
+        <material name="Red"/>
+      </visual>
+      <collision>
+        <origin rpy="0 0 0 " xyz="0 0 0" />
+        <geometry>
+          	<mesh filename="package://mrs_description/meshes/hokuyo.dae"/>
+        </geometry>
+      </collision>
+      <inertial>
+        <mass value="1e-5" />
+        <origin xyz="0 0 0" rpy="0 0 0"/>
+        <inertia ixx="1e-6" ixy="0" ixz="0" iyy="1e-6" iyz="0" izz="1e-6" />
+      </inertial>
+    </link>
+    <gazebo reference="${instance}_${prefix}_laser_link">
+      <sensor type="gpu_ray" name="${instance}_${prefix}_lasersensor">
+        <pose>0 0 0 0 0 0</pose>
+        <visualize>false</visualize>
+        <update_rate>40</update_rate>
+        <ray>
+          <scan>
+            <horizontal>
+              <samples>720</samples>
+              <resolution>1</resolution>
+              <min_angle>-1.570796</min_angle>
+              <max_angle>1.570796</max_angle>
+            </horizontal>
+          </scan>
+          <range>
+            <min>0.10</min>
+            <max>30.0</max>
+            <resolution>0.01</resolution>
+          </range>
+        </ray>
+        <plugin name="gazebo_ros_head_hokuyo_controller" filename="libgazebo_ros_gpu_laser.so">
+          <topicName>/mrs/${instance}_${prefix}_lasersensor</topicName>
+          <frameName>${instance}_${prefix}_laser_link</frameName>
+        </plugin>
+      </sensor>
+    </gazebo>
+	</xacro:macro>
 	<xacro:macro name="SMRadprobe" params="parent prefix reflect instance">
 		<joint name="${instance}_${prefix}_SMRadprobe_joint" type="fixed">

Commit message: teleop and power base with camera, laser and imu

File: mrs_description/robots/power_base.xacro (robot description, xacro)
@@ -20,5 +20,4 @@
   <xacro:Ball_bearing mass="0.1" instance="3" dia="0.05" x="0.05" y="-0.05" z="-0.05" parent="base_link"/>
   <xacro:Ball_bearing mass="0.1" instance="4" dia="0.05" x="-0.05" y="-0.05" z="-0.05" parent="base_link"/>
-<!--
   <gazebo>
     <plugin name="gazebo_ros_controller_manager" filename="libgazebo_ros_control.so">
@@ -26,5 +25,5 @@
     </plugin>
     <plugin name="object_controller" filename="libgazebo_ros_planar_move.so">
-      <commandTopic>cmd_vel</commandTopic>
+      <commandTopic>/mrs/cmd_vel</commandTopic>
       <odometryTopic>odom</odometryTopic>
       <odometryFrame>odom</odometryFrame>
@@ -33,4 +32,3 @@
     </plugin>
   </gazebo>
--->
 </robot>

File: mrs_description/urdf/power_base/base.urdf.xacro (robot description, xacro)
@@ -82,14 +82,10 @@
   </gazebo>
   </xacro:macro>
-<xacro:Camera parent="base_link_support" prefix="base" x="0.15"
-y="0" z="0.27" instance="1" />
-<xacro:Camera parent="base_link_support" prefix="base" x="0"
-y="0.15" z="0.27" instance="2" />
-<xacro:Camera parent="base_link_support" prefix="base" x="-0.15"
-y="0" z="0.27" instance="3" />
-<xacro:Camera parent="base_link_support" prefix="base" x="0"
-y="-0.15" z="0.27" instance="4" />
-<xacro:Laser parent="base_link_support" prefix="base" x="0"
-y="0" z="0.31" instance="1" />
+<xacro:Camera parent="base_link_support" prefix="base" x="0.15" y="0" z="0.27" instance="1" />
+<xacro:Camera parent="base_link_support" prefix="base" x="0" y="0.15" z="0.27" instance="2" />
+<xacro:Camera parent="base_link_support" prefix="base" x="-0.15" y="0" z="0.27" instance="3" />
+<xacro:Camera parent="base_link_support" prefix="base" x="0" y="-0.15" z="0.27" instance="4" />
+<xacro:Laser parent="base_link_support" prefix="base" x="0" y="0" z="0.31" instance="1" />
+<xacro:IMU parent="base_link_support" prefix="base" x="0.1" y="0.1" z="0.31"  />
 <!--
    <xacro:ball_bearing mass="0.1" instance="1" dia="0.05" x="0" y="0" z="-0.05" parent="base_link"/>

File: mrs_description/urdf/power_base/sm_other.urdf.xacro (robot description, xacro)
@@ -39,5 +39,6 @@
       <material>Gazebo/Red</material>
       <sensor type="camera" name="${instance}_${prefix}_camera">
-      <update_rate>30.0</update_rate>
+        <always_on>true</always_on>
+        <update_rate>30.0</update_rate>
         <camera name="${instance}_${prefix}_camera">
           <horizontal_fov>1.3962634</horizontal_fov>
@@ -53,6 +54,8 @@
         </camera>
         <plugin name="camera_controller" filename="libgazebo_ros_camera.so">
+<!--
           <alwaysOn>true</alwaysOn>
-          <updateRate>0.0</updateRate>
+          <updateRate>30.0</updateRate>
+-->
           <cameraName>mrs/${instance}_${prefix}_camera</cameraName>
           <imageTopicName>image_raw</imageTopicName>
@@ -69,4 +72,49 @@
     </gazebo>
 	</xacro:macro>
+  <xacro:macro name="IMU" params="parent prefix x y z">
+    <joint name="${prefix}_imu_joint" type="fixed">
+      <axis xyz="1 0 0" />
+      <parent link="${parent}" />
+      <child link="${prefix}_imu_link" />
+      <origin rpy="0 0 0" xyz="${x} ${y} ${z}" />
+    </joint>
+    <link name="${prefix}_imu_link">
+      <visual>
+        <geometry>
+          	<box size="0.001 0.001 0.001"/>
+        </geometry>
+        <origin rpy="0 0 0 " xyz="0 0 0" />
+        <material name="Red"/>
+      </visual>
+      <collision>
+        <origin rpy="0 0 0 " xyz="0 0 0" />
+        <geometry>
+          	<box size="0.001 0.001 0.001"/>
+        </geometry>
+      </collision>
+      <inertial>
+        <mass value="1e-5" />
+        <origin xyz="0 0 0" rpy="0 0 0"/>
+        <inertia ixx="1e-6" ixy="0" ixz="0" iyy="1e-6" iyz="0" izz="1e-6" />
+      </inertial>
+    </link>
+    <gazebo>
+<!--
+      <sensor name="Vilma_IMU" type="imu">
+        <pose>0 0 0 0 0 0</pose>
+        <imu>
+          <topic>__default_topic__</topic>
+        </imu>
+        <always_on>1</always_on>
+        <update_rate>30</update_rate>
+      </sensor>
+-->
+      <plugin filename="libgazebo_ros_imu.so" name="imu_en_ros">
+        <bodyName>${prefix}_imu_link</bodyName>
+        <robotNamespace>mrs</robotNamespace>
+        <topicName>${prefix}_IMU</topicName>
+      </plugin>
+    </gazebo>
+  </xacro:macro>
 	<xacro:macro name="Laser" params="parent prefix x y z instance">
     <joint name="${instance}_${prefix}_laser_joint" type="fixed">
@@ -155,12 +203,12 @@
 			</visual>
 		</link>
-	<gazebo reference="${instance}_${prefix}_rad_pole">
-		<material>Gazebo/Red</material>
-		<selfCollide>false</selfCollide>
-	</gazebo>
-	<gazebo reference="${instance}_${prefix}_rad">
-		<material>Gazebo/Black</material>
-		<selfCollide>false</selfCollide>
-	</gazebo>
+    <gazebo reference="${instance}_${prefix}_rad_pole">
+      <material>Gazebo/Red</material>
+      <selfCollide>false</selfCollide>
+    </gazebo>
+    <gazebo reference="${instance}_${prefix}_rad">
+      <material>Gazebo/Black</material>
+      <selfCollide>false</selfCollide>
+    </gazebo>
 	</xacro:macro>
 	<xacro:macro name="SMHand" params="parent prefix reflect instance">
@@ -237,20 +285,20 @@
 			</visual>
 		</link>
-	<gazebo reference="${instance}_${prefix}_gripper_pole">
-		<material>Gazebo/Grey</material>
-		<selfCollide>false</selfCollide>
-	</gazebo>
-	<gazebo reference="${instance}_${prefix}_left_gripper">
-		<material>Gazebo/Grey</material>
-		<selfCollide>false</selfCollide>
-	</gazebo>
-	<gazebo reference="${instance}_${prefix}_left_tip">
-		<material>Gazebo/Grey</material>
-		<selfCollide>false</selfCollide>
-	</gazebo>
-	<gazebo reference="${instance}_${prefix}_right_gripper">
-		<material>Gazebo/Grey</material>
-		<selfCollide>false</selfCollide>
-	</gazebo>
+    <gazebo reference="${instance}_${prefix}_gripper_pole">
+      <material>Gazebo/Grey</material>
+      <selfCollide>false</selfCollide>
+    </gazebo>
+    <gazebo reference="${instance}_${prefix}_left_gripper">
+      <material>Gazebo/Grey</material>
+      <selfCollide>false</selfCollide>
+    </gazebo>
+    <gazebo reference="${instance}_${prefix}_left_tip">
+      <material>Gazebo/Grey</material>
+      <selfCollide>false</selfCollide>
+    </gazebo>
+    <gazebo reference="${instance}_${prefix}_right_gripper">
+      <material>Gazebo/Grey</material>
+      <selfCollide>false</selfCollide>
+    </gazebo>
 	</xacro:macro>
-	</robot>
+</robot>
