Commit message: Working on simplified MRS for reconfiguration

File: mrs_description/robots/W2M.xacro (robot description, xacro)
@@ -1,13 +1,13 @@
 <?xml version="1.0"?>
 <robot name="mrs" xmlns:xacro="http://www.ros.org/wiki/xacro">
-	<!-- Constants for robot -->
-	<xacro:include filename="$(find mrs_description)/urdf/common_mrs.xacro" />
-	<!-- Import all Gazebo-customization elements, including Gazebo colors -->
-	<xacro:include filename="$(find mrs_description)/urdf/power_base/ball_bearing.urdf.xacro" />
-	<xacro:include filename="$(find mrs_description)/urdf/JM/jm.xacro" />
-	<xacro:include filename="$(find mrs_description)/urdf/PCM/pcm.xacro" />
-	<!-- Used for fixing robot to Gazebo 'base_link' -->
-	<link name="world" >
-		<inertial>
+  <!-- Constants for robot -->
+  <xacro:include filename="$(find mrs_description)/urdf/common_mrs.xacro" />
+  <!-- Import all Gazebo-customization elements, including Gazebo colors -->
+  <xacro:include filename="$(find mrs_description)/urdf/power_base/ball_bearing.urdf.xacro" />
+  <xacro:include filename="$(find mrs_description)/urdf/JM/jm.xacro" />
+  <xacro:include filename="$(find mrs_description)/urdf/PCM/pcm.xacro" />
+  <!-- Used for fixing robot to Gazebo 'base_link' -->
+  <link name="world" >
+    <inertial>
         <mass value="0.1"/>
         <origin xyz="0 0 0" rpy="0 0 0"/>
@@ -28,55 +28,53 @@
       </collision>
     </link>
-	<joint name="fixed" type="fixed">
-		<axis xyz="1 0 0 " />
-		<origin xyz="0 0 0.05" rpy="0 ${-pi/2} 0" />
-		<!-- <origin xyz="0 0 0.1" rpy="0 0 0" /> -->
-		<parent link="world" />
-		<child link="base_footprint" />
-	</joint>
-	<!-- Fictitious Base Link is a fictitious link(frame) that is on the ground below
-		base_link origin, Dummy link-->
-	<link name="base_footprint">
-			<mass value="1.0" />
-			<visual>
-				<geometry>
-					<box size="0.07 0.07 0.14" />
-				</geometry>
-				<material name="Blue">
-				</material>
-			</visual>
-			<collision>
-				<geometry>
-					<box size="0.05 0.05 0.04" />
-				</geometry>
-			</collision>
-			<xacro:default_inertial mass="0.15" I_tensor="8.166e-4"/>
-	</link>
-	  	<gazebo reference="base_footprint">
-		<material>Gazebo/Blue</material>
-		<selfCollide>false</selfCollide>
-	</gazebo>
-	<xacro:JM3_prismatic name="JM" prefix="W1" instance="1"  parent="W1_PCmodule" reflect="1" shift="0.035"/>
-	<xacro:PcModule_solid parent="base_footprint" prefix="W1" reflect="-1" />
-	<xacro:PcModule_solid parent="base_footprint" prefix="W2" reflect="1" />
-	<xacro:JM3_prismatic name="JM1" prefix="W1" instance="2"  parent="W2_PCmodule" reflect="-1" shift="0.035"/>
+  <joint name="fixed" type="fixed">
+    <axis xyz="1 0 0 " />
+    <origin xyz="0 0 0.05" rpy="0 ${-pi/2} 0" />
+    <!-- <origin xyz="0 0 0.1" rpy="0 0 0" /> -->
+    <parent link="world" />
+    <child link="base_footprint" />
+  </joint>
+  <!-- Fictitious Base Link is a fictitious link(frame) that is on the ground below
+    base_link origin, Dummy link-->
+  <link name="base_footprint">
+      <mass value="1.0" />
+      <visual>
+        <geometry>
+          <box size="0.07 0.07 0.14" />
+        </geometry>
+        <material name="Blue">
+        </material>
+      </visual>
+      <collision>
+        <geometry>
+          <box size="0.05 0.05 0.04" />
+        </geometry>
+      </collision>
+      <xacro:default_inertial mass="0.15" I_tensor="8.166e-4"/>
+  </link>
+      <gazebo reference="base_footprint">
+    <material>Gazebo/Blue</material>
+    <selfCollide>false</selfCollide>
+  </gazebo>
+  <xacro:JM3_solid name="JM" prefix="W1" instance="1"  parent="W1_PCmodule" reflect="1" shift="0.035"/>
+  <xacro:PcModule_solid parent="base_footprint" prefix="W1" reflect="-1" />
+  <xacro:PcModule_solid parent="base_footprint" prefix="W2" reflect="1" />
+  <xacro:JM3_solid name="JM1" prefix="W1" instance="2"  parent="W2_PCmodule" reflect="-1" shift="0.035"/>
+<!--
   <xacro:Ball_bearing mass="0.1" instance="1" dia="0.01" x="-0.045" y="0.0" z="-0.2" parent="base_footprint"/>
   <xacro:Ball_bearing mass="0.1" instance="2" dia="0.01" x="-0.045" y="0.0" z="0.2" parent="base_footprint"/>
-<!--
-	<xacro:Ball_bearing mass="0.1" instance="1" dia="0.05" x="-0.035" y="0" z="0.035" parent="base_footprint"/>
-	<xacro:Ball_bearing mass="0.1" instance="2" dia="0.05" x="-0.035" y="0" z="0.070" parent="base_footprint"/>
 -->
-	<!-- ros_control plugin -->
-	<gazebo>
-		<plugin name="mrs_ros_control" filename="libgazebo_ros_control.so">
-			<controlPeriod>0.001</controlPeriod>
-			<robotNamespace>/mrs</robotNamespace>
-		</plugin>
-	  <plugin name="object_controller" filename="libgazebo_ros_planar_move.so">
-      <commandTopic>cmd_vel</commandTopic>
+  <xacro:Ball_bearing mass="0.1" instance="1" dia="0.01" x="-0.055" y="0" z="-0.07" parent="base_footprint"/>
+  <xacro:Ball_bearing mass="0.1" instance="2" dia="0.01" x="-0.055" y="0" z="0.07" parent="base_footprint"/>
+  <gazebo>
+    <plugin name="gazebo_ros_controller_manager" filename="libgazebo_ros_control.so">
+      <robotNamespace>/mrs</robotNamespace>
+    </plugin>
+    <plugin name="object_controller" filename="libgazebo_ros_planar_move.so">
+      <commandTopic>/mrs/cmd_vel</commandTopic>
       <odometryTopic>odom</odometryTopic>
       <odometryFrame>odom</odometryFrame>
       <odometryRate>20.0</odometryRate>
-      <robotBaseFrame>world</robotBaseFrame>
+      <robotBaseFrame>base_footprint</robotBaseFrame>
     </plugin>
   </gazebo>

File: mrs_description/robots/power_base.xacro (robot description, xacro)
@@ -16,8 +16,10 @@
   <!-- foot for arm-->
   <xacro:power_base name="base"/>
+<!--
   <xacro:Ball_bearing mass="0.1" instance="1" dia="0.05" x="0.05" y="0.05" z="-0.05" parent="base_link"/>
   <xacro:Ball_bearing mass="0.1" instance="2" dia="0.05" x="-0.05" y="0.05" z="-0.05" parent="base_link"/>
   <xacro:Ball_bearing mass="0.1" instance="3" dia="0.05" x="0.05" y="-0.05" z="-0.05" parent="base_link"/>
   <xacro:Ball_bearing mass="0.1" instance="4" dia="0.05" x="-0.05" y="-0.05" z="-0.05" parent="base_link"/>
+-->
   <gazebo>
     <plugin name="gazebo_ros_controller_manager" filename="libgazebo_ros_control.so">

File: mrs_description/urdf/JM/jm.xacro (robot description, xacro)
@@ -1,393 +1,393 @@
 <?xml version="1.0"?>
 <robot name="mrs" xmlns:xacro="http://www.ros.org/wiki/xacro">
-	<!-- Constants for robot -->
-	<xacro:include filename="$(find mrs_description)/urdf/common_mrs.xacro" />
-	<!-- Import all Gazebo-customization elements, including Gazebo colors -->
-	<xacro:include filename="$(find mrs_description)/urdf/JM/jm.gazebo.xacro" />
-	<!-- Import Rviz colors -->
-	<xacro:include filename="$(find mrs_description)/urdf/materials.urdf.xacro" />
+  <!-- Constants for robot -->
+  <xacro:include filename="$(find mrs_description)/urdf/common_mrs.xacro" />
+  <!-- Import all Gazebo-customization elements, including Gazebo colors -->
+  <xacro:include filename="$(find mrs_description)/urdf/JM/jm.gazebo.xacro" />
+  <!-- Import Rviz colors -->
+  <xacro:include filename="$(find mrs_description)/urdf/materials.urdf.xacro" />
 <macro name="JM1" params="name prefix instance parent">
-	<!-- Links -->
-	<create_link name="j1_link" color="Blue" mesh="${j1_mesh}"
-		cog="${j1_cog}" mass="${j1_mass}" instance="${instance}" prefix="${prefix}">
-		<j1_inertia />
-	</create_link>
-	<create_link_no_collision name="j2_link" color="Blue" mesh="${j2_mesh}"
-		cog="${j2_cog}" mass="${j2_mass}" instance="${instance}" prefix="${prefix}">
-		<j2_inertia />
-	</create_link_no_collision>
-	<create_link_no_collision name="j3_link" color="Blue" mesh="${j3_mesh}"
-		cog="${j3_cog}" mass="${j3_mass}" instance="${instance}" prefix="${prefix}">
-		<j3_inertia />
-	</create_link_no_collision>
-	<create_link name="w1_link" color="Blue" mesh="${w1_mesh}"
-		cog="${w1_cog}" mass="${w1_mass}" instance="${instance}" prefix="${prefix}">
-		<w1_inertia />
-	</create_link>
-	<!-- Joints -->
-	<joint name="${instance}_${prefix}_j3" type="fixed">
-		<child link="${instance}_${prefix}_w1_link" />
-		<parent link="${parent}" />
-		<axis xyz="0 0 1 " />
-		<origin xyz="0 0 0.01" rpy="0 ${-pi/2} 0" />
-<!--
-		<limit lower="${-pi/2}" upper="${pi/2}" effort="${max_effort}"
-			velocity="${max_velocity}" />
-		<dynamics damping="${j3_damping}" />
--->
-	</joint>
-	<joint name="${instance}_${prefix}_j2_fixed" type="fixed">
-		<child link="${instance}_${prefix}_j3_link" />
-		<parent link="${instance}_${prefix}_w1_link" />
-		<origin xyz="0.045 0 0" rpy="0 0 ${pi/2}" />
-	</joint>
-	<joint name="${instance}_${prefix}_j2" type="revolute">
-		<child link="${instance}_${prefix}_j1_link" />
-		<parent link="${instance}_${prefix}_j3_link" />
-		<axis xyz="1 0 0 " />
-		<origin xyz="0 0 0" rpy="0 ${-pi/2} 0" />
-		<limit lower="${-pi/2}" upper="${pi/2}" effort="${max_effort}"
-			velocity="${max_velocity}" />
-		<dynamics damping="${j2_damping}" />
-	</joint>
-	<joint name="${instance}_${prefix}_j1" type="revolute">
-		<child link="${instance}_${prefix}_j2_link" />
-		<parent link="${instance}_${prefix}_j1_link" />
-		<axis xyz="0 0 1 " />
-		<origin xyz="0 -0.058 0" rpy="${pi/2} 0 0" />
-		<limit lower="${-pi/2}" upper="${pi/2}" effort="${max_effort}"
-			velocity="${max_velocity}" />
-		<dynamics damping="${j3_damping}" />
-	</joint>
-		<!-- Transmissions -->
-	<simple_transmission joint="${instance}_${prefix}_j1" />
-	<simple_transmission joint="${instance}_${prefix}_j2" />
-<!--
-	<simple_transmission joint="${instance}_${prefix}_j3" />
--->
-		<!-- Gazebo  -->
-	<xacro:JMG name="${name}_gazebo" prefix="${prefix}" instance="${instance}" />
-	</macro>
+  <!-- Links -->
+  <create_link name="j1_link" color="Blue" mesh="${j1_mesh}"
+    cog="${j1_cog}" mass="${j1_mass}" instance="${instance}" prefix="${prefix}">
+    <j1_inertia />
+  </create_link>
+  <create_link_no_collision name="j2_link" color="Blue" mesh="${j2_mesh}"
+    cog="${j2_cog}" mass="${j2_mass}" instance="${instance}" prefix="${prefix}">
+    <j2_inertia />
+  </create_link_no_collision>
+  <create_link_no_collision name="j3_link" color="Blue" mesh="${j3_mesh}"
+    cog="${j3_cog}" mass="${j3_mass}" instance="${instance}" prefix="${prefix}">
+    <j3_inertia />
+  </create_link_no_collision>
+  <create_link name="w1_link" color="Blue" mesh="${w1_mesh}"
+    cog="${w1_cog}" mass="${w1_mass}" instance="${instance}" prefix="${prefix}">
+    <w1_inertia />
+  </create_link>
+  <!-- Joints -->
+  <joint name="${instance}_${prefix}_j3" type="fixed">
+    <child link="${instance}_${prefix}_w1_link" />
+    <parent link="${parent}" />
+    <axis xyz="0 0 1 " />
+    <origin xyz="0 0 0.01" rpy="0 ${-pi/2} 0" />
+<!--
+    <limit lower="${-pi/2}" upper="${pi/2}" effort="${max_effort}"
+      velocity="${max_velocity}" />
+    <dynamics damping="${j3_damping}" />
+-->
+  </joint>
+  <joint name="${instance}_${prefix}_j2_fixed" type="fixed">
+    <child link="${instance}_${prefix}_j3_link" />
+    <parent link="${instance}_${prefix}_w1_link" />
+    <origin xyz="0.045 0 0" rpy="0 0 ${pi/2}" />
+  </joint>
+  <joint name="${instance}_${prefix}_j2" type="revolute">
+    <child link="${instance}_${prefix}_j1_link" />
+    <parent link="${instance}_${prefix}_j3_link" />
+    <axis xyz="1 0 0 " />
+    <origin xyz="0 0 0" rpy="0 ${-pi/2} 0" />
+    <limit lower="${-pi/2}" upper="${pi/2}" effort="${max_effort}"
+      velocity="${max_velocity}" />
+    <dynamics damping="${j2_damping}" />
+  </joint>
+  <joint name="${instance}_${prefix}_j1" type="revolute">
+    <child link="${instance}_${prefix}_j2_link" />
+    <parent link="${instance}_${prefix}_j1_link" />
+    <axis xyz="0 0 1 " />
+    <origin xyz="0 -0.058 0" rpy="${pi/2} 0 0" />
+    <limit lower="${-pi/2}" upper="${pi/2}" effort="${max_effort}"
+      velocity="${max_velocity}" />
+    <dynamics damping="${j3_damping}" />
+  </joint>
+    <!-- Transmissions -->
+  <simple_transmission joint="${instance}_${prefix}_j1" />
+  <simple_transmission joint="${instance}_${prefix}_j2" />
+<!--
+  <simple_transmission joint="${instance}_${prefix}_j3" />
+-->
+    <!-- Gazebo  -->
+  <xacro:JMG name="${name}_gazebo" prefix="${prefix}" instance="${instance}" />
+  </macro>
 <macro name="JM1_kinematic" params="name prefix instance parent">
-	<!-- Links -->
-	<create_link name="j1_link" color="Grey" mesh="${j1_mesh}"
-		cog="${j1_cog}" mass="${j1_mass}" instance="${instance}" prefix="${prefix}">
-		<j1_inertia />
-	</create_link>
-<!--
-	<create_link name="j2_link" color="Grey" mesh="${j2_mesh}"
-		cog="${j2_cog}" mass="${j2_mass}" instance="${instance}" prefix="${prefix}">
-		<j2_inertia />
-	</create_link>
--->
-	<link name="1_L1_j2_link">
-			<visual>
-				<geometry>
-					<cylinder length="0.15" radius=".03" />
-				</geometry>
-				<origin rpy="0 0 0 " xyz="0 0 0" />
-				<material name="Gray">
-					<color rgba=".7 .7 .7 1" />
-				</material>
-			</visual>
-			<collision>
-				<geometry>
-					<cylinder length="0.06" radius=".01" />
-				</geometry>
-			</collision>
-		</link>
-<!--
-	<create_link_no_collision name="j3_link" color="Blue" mesh="${j3_mesh}"
-		cog="${j3_cog}" mass="${j3_mass}" instance="${instance}" prefix="${prefix}">
-		<j3_inertia />
-	</create_link_no_collision>
--->
-	<create_link name="w1_link" color="Black" mesh="${w1_mesh}"
-		cog="${w1_cog}" mass="${w1_mass}" instance="${instance}" prefix="${prefix}">
-		<w1_inertia />
-	</create_link>
-	<!-- Joints -->
-	<joint name="${instance}_${prefix}_j3" type="revolute">
-		<child link="${instance}_${prefix}_w1_link" />
-		<parent link="${parent}" />
-		<axis xyz="1 0 0 " />
-		<origin xyz="0 0 0.01" rpy="0 ${-pi/2} 0" />
-		<limit lower="${-pi}" upper="${pi}" effort="${max_effort}"
-			velocity="${max_velocity}" />
-		<dynamics damping="${j3_damping}" />
-	</joint>
-<!--
-	<joint name="${instance}_${prefix}_j2_fixed" type="fixed">
-		<child link="${instance}_${prefix}_j3_link" />
-		<parent link="${instance}_${prefix}_w1_link" />
-		<origin xyz="0.045 0 0" rpy="0 0 ${pi/2}" />
-	</joint>
--->
-	<joint name="${instance}_${prefix}_j2" type="revolute">
-		<child link="${instance}_${prefix}_j1_link" />
-		<parent link="${instance}_${prefix}_w1_link" />
-		<axis xyz="1 0 0 " />
-		<origin xyz="0.045 0 0" rpy="0 ${pi/2} ${pi/2}" />
-		<limit lower="${-pi/2}" upper="${pi/2}" effort="${max_effort}"
-			velocity="${max_velocity}" />
-		<dynamics damping="${j2_damping}" />
-	</joint>
-	<joint name="${instance}_${prefix}_j1" type="revolute">
-		<child link="${instance}_${prefix}_j2_link" />
-		<parent link="${instance}_${prefix}_j1_link" />
-		<axis xyz="0 1 0 " />
-		<origin xyz="0 -0.125 0" rpy="${pi/2} 0 0" />
-		<limit lower="${-pi/2}" upper="${pi/2}" effort="${max_effort}"
-			velocity="${max_velocity}" />
-		<dynamics damping="${j3_damping}" />
-	</joint>
-		<!-- Transmissions -->
-	<simple_transmission joint="${instance}_${prefix}_j1" />
-	<simple_transmission joint="${instance}_${prefix}_j2" />
-	<simple_transmission joint="${instance}_${prefix}_j3" />
-		<!-- Gazebo  -->
-	<xacro:JMG name="${name}_gazebo" prefix="${prefix}" instance="${instance}" />
-	</macro>
+  <!-- Links -->
+  <create_link name="j1_link" color="Grey" mesh="${j1_mesh}"
+    cog="${j1_cog}" mass="${j1_mass}" instance="${instance}" prefix="${prefix}">
+    <j1_inertia />
+  </create_link>
+<!--
+  <create_link name="j2_link" color="Grey" mesh="${j2_mesh}"
+    cog="${j2_cog}" mass="${j2_mass}" instance="${instance}" prefix="${prefix}">
+    <j2_inertia />
+  </create_link>
+-->
+  <link name="1_L1_j2_link">
+      <visual>
+        <geometry>
+          <cylinder length="0.15" radius=".03" />
+        </geometry>
+        <origin rpy="0 0 0 " xyz="0 0 0" />
+        <material name="Gray">
+          <color rgba=".7 .7 .7 1" />
+        </material>
+      </visual>
+      <collision>
+        <geometry>
+          <cylinder length="0.06" radius=".01" />
+        </geometry>
+      </collision>
+    </link>
+<!--
+  <create_link_no_collision name="j3_link" color="Blue" mesh="${j3_mesh}"
+    cog="${j3_cog}" mass="${j3_mass}" instance="${instance}" prefix="${prefix}">
+    <j3_inertia />
+  </create_link_no_collision>
+-->
+  <create_link name="w1_link" color="Black" mesh="${w1_mesh}"
+    cog="${w1_cog}" mass="${w1_mass}" instance="${instance}" prefix="${prefix}">
+    <w1_inertia />
+  </create_link>
+  <!-- Joints -->
+  <joint name="${instance}_${prefix}_j3" type="revolute">
+    <child link="${instance}_${prefix}_w1_link" />
+    <parent link="${parent}" />
+    <axis xyz="1 0 0 " />
+    <origin xyz="0 0 0.01" rpy="0 ${-pi/2} 0" />
+    <limit lower="${-pi}" upper="${pi}" effort="${max_effort}"
+      velocity="${max_velocity}" />
+    <dynamics damping="${j3_damping}" />
+  </joint>
+<!--
+  <joint name="${instance}_${prefix}_j2_fixed" type="fixed">
+    <child link="${instance}_${prefix}_j3_link" />
+    <parent link="${instance}_${prefix}_w1_link" />
+    <origin xyz="0.045 0 0" rpy="0 0 ${pi/2}" />
+  </joint>
+-->
+  <joint name="${instance}_${prefix}_j2" type="revolute">
+    <child link="${instance}_${prefix}_j1_link" />
+    <parent link="${instance}_${prefix}_w1_link" />
+    <axis xyz="1 0 0 " />
+    <origin xyz="0.045 0 0" rpy="0 ${pi/2} ${pi/2}" />
+    <limit lower="${-pi/2}" upper="${pi/2}" effort="${max_effort}"
+      velocity="${max_velocity}" />
+    <dynamics damping="${j2_damping}" />
+  </joint>
+  <joint name="${instance}_${prefix}_j1" type="revolute">
+    <child link="${instance}_${prefix}_j2_link" />
+    <parent link="${instance}_${prefix}_j1_link" />
+    <axis xyz="0 1 0 " />
+    <origin xyz="0 -0.125 0" rpy="${pi/2} 0 0" />
+    <limit lower="${-pi/2}" upper="${pi/2}" effort="${max_effort}"
+      velocity="${max_velocity}" />
+    <dynamics damping="${j3_damping}" />
+  </joint>
+    <!-- Transmissions -->
+  <simple_transmission joint="${instance}_${prefix}_j1" />
+  <simple_transmission joint="${instance}_${prefix}_j2" />
+  <simple_transmission joint="${instance}_${prefix}_j3" />
+    <!-- Gazebo  -->
+  <xacro:JMG name="${name}_gazebo" prefix="${prefix}" instance="${instance}" />
+  </macro>
 <macro name="JM2" params="name prefix instance parent reflect shift shift2">
-	<create_link name="j1_link" color="Blue" mesh="${j1_mesh}"
-		cog="${j1_cog}" mass="${j1_mass}" instance="${instance}" prefix="${prefix}">
-		<j1_inertia />
-	</create_link>
-	<create_link_no_collision name="j2_link" color="Blue" mesh="${j2_mesh}"
-		cog="${j2_cog}" mass="${j2_mass}" instance="${instance}" prefix="${prefix}">
-		<j2_inertia />
-	</create_link_no_collision>
-	<create_link_no_collision name="j3_link" color="Blue" mesh="${j3_mesh}"
-		cog="${j3_cog}" mass="${j3_mass}" instance="${instance}" prefix="${prefix}">
-		<j3_inertia />
-	</create_link_no_collision>
-	<create_link name="w1_link" color="Blue" mesh="${w1_mesh}"
-		cog="${w1_cog}" mass="${w1_mass}" instance="${instance}" prefix="${prefix}">
-		<w1_inertia />
-	</create_link>
-	<joint name="${instance}_${prefix}_j3" type="revolute">
-		<child link="${instance}_${prefix}_w1_link" />
-		<parent link="${instance}_${prefix}_j3_link" />
-		<axis xyz="1 0 0" />
-		<origin xyz="0 0.05 0" rpy="0 0 ${-pi/2}" />
-		<limit lower="${-pi}" upper="${pi}" effort="${max_effort}"
-			velocity="${max_velocity}" />
-		<dynamics damping="${j1_damping}" />
-	</joint>
-	<joint name="${instance}_${prefix}_j2" type="revolute">
-		<child link="${instance}_${prefix}_j3_link" />
-		<parent link="${instance}_${prefix}_j1_link" />
-		<axis xyz="0 0 1 " />
-		<origin xyz="0 0 0" rpy="0 ${pi/2} 0" />
-		<limit lower="${-pi/2}" upper="${pi/2}" effort="${max_effort}"
-			velocity="${max_velocity}" />
-		<dynamics damping="${j2_damping}" />
-	</joint>
-	<joint name="${instance}_${prefix}_j2_fixed" type="fixed">
-		<child link="${instance}_${prefix}_j1_link" />
-		<parent link="${instance}_${prefix}_j2_link" />
-		<axis xyz="1 0 0 " />
-		<origin xyz="0 0 0.058" rpy="${pi/2} 0 ${pi/2}" />
-	</joint>
-	<joint name="${instance}_${prefix}_j1" type="revolute">
-		<child link="${instance}_${prefix}_j2_link" />
-		<parent link="${parent}" />
-		<axis xyz="0 0 1 " />
-		<origin xyz="${shift*reflect} 0 ${shift*shift2}" rpy="0 ${reflect*pi/2} 0" />
-		<limit lower="0" upper="${pi}" effort="${max_effort}"
-			velocity="${max_velocity}" />
-		<dynamics damping="${j3_damping}" />
-	</joint>
-		<!-- Transmissions -->
-	<simple_transmission joint="${instance}_${prefix}_j1" />
-	<simple_transmission joint="${instance}_${prefix}_j2" />
-	<simple_transmission joint="${instance}_${prefix}_j3" />
-	<!-- Gazebo  -->
-	<xacro:JMG name="${name}_gazebo" prefix="${prefix}" instance="${instance}" />
-	</macro>
+  <create_link name="j1_link" color="Blue" mesh="${j1_mesh}"
+    cog="${j1_cog}" mass="${j1_mass}" instance="${instance}" prefix="${prefix}">
+    <j1_inertia />
+  </create_link>
+  <create_link_no_collision name="j2_link" color="Blue" mesh="${j2_mesh}"
+    cog="${j2_cog}" mass="${j2_mass}" instance="${instance}" prefix="${prefix}">
+    <j2_inertia />
+  </create_link_no_collision>
+  <create_link_no_collision name="j3_link" color="Blue" mesh="${j3_mesh}"
+    cog="${j3_cog}" mass="${j3_mass}" instance="${instance}" prefix="${prefix}">
+    <j3_inertia />
+  </create_link_no_collision>
+  <create_link name="w1_link" color="Blue" mesh="${w1_mesh}"
+    cog="${w1_cog}" mass="${w1_mass}" instance="${instance}" prefix="${prefix}">
+    <w1_inertia />
+  </create_link>
+  <joint name="${instance}_${prefix}_j3" type="revolute">
+    <child link="${instance}_${prefix}_w1_link" />
+    <parent link="${instance}_${prefix}_j3_link" />
+    <axis xyz="1 0 0" />
+    <origin xyz="0 0.05 0" rpy="0 0 ${-pi/2}" />
+    <limit lower="${-pi}" upper="${pi}" effort="${max_effort}"
+      velocity="${max_velocity}" />
+    <dynamics damping="${j1_damping}" />
+  </joint>
+  <joint name="${instance}_${prefix}_j2" type="revolute">
+    <child link="${instance}_${prefix}_j3_link" />
+    <parent link="${instance}_${prefix}_j1_link" />
+    <axis xyz="0 0 1 " />
+    <origin xyz="0 0 0" rpy="0 ${pi/2} 0" />
+    <limit lower="${-pi/2}" upper="${pi/2}" effort="${max_effort}"
+      velocity="${max_velocity}" />
+    <dynamics damping="${j2_damping}" />
+  </joint>
+  <joint name="${instance}_${prefix}_j2_fixed" type="fixed">
+    <child link="${instance}_${prefix}_j1_link" />
+    <parent link="${instance}_${prefix}_j2_link" />
+    <axis xyz="1 0 0 " />
+    <origin xyz="0 0 0.058" rpy="${pi/2} 0 ${pi/2}" />
+  </joint>
+  <joint name="${instance}_${prefix}_j1" type="revolute">
+    <child link="${instance}_${prefix}_j2_link" />
+    <parent link="${parent}" />
+    <axis xyz="0 0 1 " />
+    <origin xyz="${shift*reflect} 0 ${shift*shift2}" rpy="0 ${reflect*pi/2} 0" />
+    <limit lower="0" upper="${pi}" effort="${max_effort}"
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