Commit message: Working on simplified MRS for reconfiguration

File: mrs_description/urdf/power_base/base.urdf.xacro (robot description, xacro)
@@ -2,5 +2,5 @@
 <robot xmlns:xacro="http://www.ros.org/wiki/xacro">
 <xacro:include filename="$(find mrs_description)/urdf/power_base/ball_bearing.urdf.xacro" />
-		<!-- constants for robot -->
+    <!-- constants for robot -->
 <xacro:include filename="$(find mrs_description)/urdf/common_mrs.xacro" />
   <!-- simplified box collision geometry for base -->
@@ -9,6 +9,6 @@
   <property name="mass" value="22.0"/>
   <property name="p_baselen" value=".3" />
-	<property name="p_basewidth" value=".3" />
-	<property name="p_baseheight" value=".1" />
+  <property name="p_basewidth" value=".3" />
+  <property name="p_baseheight" value=".6" />
   <xacro:macro name="power_base" params="name">
   <link name="${name}_footprint">
@@ -34,7 +34,8 @@
   <joint name="${name}_footprint_joint" type="fixed">
     <origin xyz="0 0 0" rpy="0 0 0"/>
-    <child link="${name}_link"/>
+    <child link="${name}_link_support"/>
     <parent link="${name}_footprint"/>
   </joint>
+<!--
   <link name="${name}_link">
   <inertial>
@@ -45,5 +46,5 @@
   <visual>
     <geometry>
-      <cylinder radius="${p_basewidth+0.05}" length="${p_baseheight}" />
+      <cylinder radius="${p_basewidth}" length="${p_baseheight}" />
     </geometry>
     <material name="White">
@@ -64,8 +65,9 @@
     <parent link="${name}_link" />
   </joint>
+-->
   <link name="${name}_link_support">
     <visual>
       <geometry>
-        <box size="${p_baselen} ${p_basewidth} ${p_baseheight*6}" />
+        <box size="${p_baselen} ${p_basewidth} ${p_baseheight}" />
       </geometry>
       <material name="Orange"/>
@@ -73,5 +75,5 @@
     <collision>
       <geometry>
-        <box size="${p_baselen-0.1} ${p_basewidth-0.05} ${p_baseheight*6-0.05}" />
+        <box size="${p_baselen-0.1} ${p_basewidth-0.05} ${p_baseheight-0.05}" />
       </geometry>
     </collision>
@@ -79,13 +81,17 @@
   </link>
   <gazebo reference="${name}_link_support">
-    <material>Gazebo/Grey</material>
+    <material>Gazebo/Orange</material>
   </gazebo>
+<xacro:Ball_bearing mass="0.1" instance="1" dia="0.05" x="0.05" y="0.05" z="-0.29" parent="${name}_link_support"/>
+<xacro:Ball_bearing mass="0.1" instance="2" dia="0.05" x="-0.05" y="0.05" z="-0.29" parent="${name}_link_support"/>
+<xacro:Ball_bearing mass="0.1" instance="3" dia="0.05" x="0.05" y="-0.05" z="-0.29" parent="${name}_link_support"/>
+<xacro:Ball_bearing mass="0.1" instance="4" dia="0.05" x="-0.05" y="-0.05" z="-0.29" parent="${name}_link_support"/>
+<xacro:Camera parent="${name}_link_support" prefix="base" x="0.15" y="0" z="0.27" instance="1" />
+<xacro:Camera parent="${name}_link_support" prefix="base" x="0" y="0.15" z="0.27" instance="2" />
+<xacro:Camera parent="${name}_link_support" prefix="base" x="-0.15" y="0" z="0.27" instance="3" />
+<xacro:Camera parent="${name}_link_support" prefix="base" x="0" y="-0.15" z="0.27" instance="4" />
+<xacro:Laser parent="${name}_link_support" prefix="base" x="0" y="0" z="0.31" instance="1" />
+<xacro:IMU parent="${name}_link_support" prefix="base" x="0.1" y="0.1" z="0.31"  />
   </xacro:macro>
-<xacro:Camera parent="base_link_support" prefix="base" x="0.15" y="0" z="0.27" instance="1" />
-<xacro:Camera parent="base_link_support" prefix="base" x="0" y="0.15" z="0.27" instance="2" />
-<xacro:Camera parent="base_link_support" prefix="base" x="-0.15" y="0" z="0.27" instance="3" />
-<xacro:Camera parent="base_link_support" prefix="base" x="0" y="-0.15" z="0.27" instance="4" />
-<xacro:Laser parent="base_link_support" prefix="base" x="0" y="0" z="0.31" instance="1" />
-<xacro:IMU parent="base_link_support" prefix="base" x="0.1" y="0.1" z="0.31"  />
 <!--
    <xacro:ball_bearing mass="0.1" instance="1" dia="0.05" x="0" y="0" z="-0.05" parent="base_link"/>
