Commit message: Updated with new robots models Moveit pkg

File: mrs_description/robots/AJM2_1.xacro (robot description, xacro)
@@ -9,11 +9,6 @@
   <xacro:include filename="$(find mrs_description)/urdf/materials.urdf.xacro" />
 -->
-  <xacro:macro name="initialising_frame" params="name child scale prefix">
+  <xacro:macro name="initialising_frame" params="name scale prefix">
   <link name="${name}">
-    <inertial>
-      <mass value="0.1"/>
-      <origin xyz="0 0 0" rpy="0 0 0"/>
-      <inertia ixx="1.0" ixy="0.0" ixz="0.0" iyy="1.0" iyz="0.0" izz="1.0"/>
-    </inertial>
     <visual>
       <origin xyz="0 0 0" rpy="0 0 0"/>
@@ -35,17 +30,17 @@
   </joint>
   <link name="${name}_dummy"/>
-  <xacro:pcm_module parent="${name}" prefix="${prefix}" instance="1" scale="${scale}" len="0.3" z="0.15" />
-  <xacro:joint_module parent="${name}" prefix="${prefix}" instance="1" scale="${scale}" rotate="0"/>
-  <xacro:sm_wheel parent="${prefix}_jm_link_1" prefix="${prefix}" instance="1" dia="${JMwidth+0.3}" length="0.2" rotate="1" x="-1" y="0"/>
-  <xacro:sm_wheel parent="${prefix}_jm_link_2" prefix="${prefix}" instance="2" dia="${JMwidth+0.3}" length="0.2" rotate="1" x="1" y="0"/>
+  <xacro:sm_wheel parent="${name}" prefix="${prefix}" instance="1" dia="${JMwidth+0.1}" length="0.1" rotate="0" x="0" y="0"/>
+  <xacro:joint_module_3DOF_vertical parent="${prefix}_sm_wheel_link_1" prefix="1" instance="1" scale="${scale}" rotate="1"/>
+  <xacro:pcm_module parent="1_jm_link_2" prefix="${prefix}" instance="1" scale="${scale}" len="0.35" z="0" x="0.18" rotate="0" />
+  <xacro:pcm_module parent="${prefix}_pcm_link_1" prefix="${prefix}" instance="2" scale="${scale}" len="0.35" z="0" x="0.35" rotate="0"/>
+  <xacro:joint_module_3DOF parent="${prefix}_pcm_link_2" prefix="2" instance="1" scale="${scale}" rotate="0"/>
+  <xacro:sm_wheel parent="2_jm_link_2" prefix="${prefix}" instance="2" dia="${JMwidth+0.1}" length="0.1" rotate="1" x="1" y="0"/>
   </xacro:macro>
-<!-- For 1 Jm mobile robot -->
-  <xacro:initialising_frame name="base_footprint" child="1_jm_link2_0" scale="1" prefix="1"/>
+<!-- For 2 JM 2 PC 2 WM mobile robot -->
+  <xacro:initialising_frame name="base_footprint" scale="1" prefix="mrs"/>
   <gazebo>
-<!--
     <plugin name="gazebo_ros_control" filename="libgazebo_ros_control.so">
       <robotNamespace>/mrs</robotNamespace>
     </plugin>
--->
   </gazebo>
 </robot>

File: mrs_description/robots/JM1W2.urdf (robot description, URDF)
Before this commit: robot mrs, 8 links, 7 joints
Links:
- link 1_pcm_link_1: mass 1 -> 0.01; geometry collision box size=0.3 0.3 0.3; visual box size=0.3 0.3 0.3
- link 1_sm_wheel_link_1: mass 0.1 -> 1; geometry collision cylinder length=0.2 radius=0.35; visual cylinder length=0.2 radius=0.35
- link 1_sm_wheel_link_2: mass 0.1 -> 1; geometry collision cylinder length=0.2 radius=0.35; visual cylinder length=0.2 radius=0.35
Joints:
- joint 1_pcm_joint_1: origin xyz=0 0 0.3 rpy=0 0 0 -> xyz=0 0 0.15 rpy=0 0 0
- joint 1_sm_wheel_joint_1: origin xyz=-0.1 0 0 rpy= 0 1.57079632679 0 -> xyz=-0.15 0 0 rpy= 0 1.57079632679 0
- joint 1_sm_wheel_joint_2: origin xyz=0.1 0 0 rpy= 0 1.57079632679 0 -> xyz=0.15 0 0 rpy= 0 1.57079632679 0

File: mrs_description/robots/JM1W2.xacro (robot description, xacro)
@@ -11,9 +11,4 @@
   <xacro:macro name="initialising_frame" params="name child scale prefix">
   <link name="${name}">
-    <inertial>
-      <mass value="0.1"/>
-      <origin xyz="0 0 0" rpy="0 0 0"/>
-      <inertia ixx="1.0" ixy="0.0" ixz="0.0" iyy="1.0" iyz="0.0" izz="1.0"/>
-    </inertial>
     <visual>
       <origin xyz="0 0 0" rpy="0 0 0"/>
@@ -35,6 +30,6 @@
   </joint>
   <link name="${name}_dummy"/>
-  <xacro:pcm_module parent="${name}" prefix="${prefix}" instance="1" scale="${scale}" len="0.3" z="0.15" />
-  <xacro:joint_module parent="${name}" prefix="${prefix}" instance="1" scale="${scale}" rotate="0"/>
+  <xacro:pcm_module parent="${name}" prefix="${prefix}" instance="1" scale="${scale}" len="0.3" z="0.15" x="0" rotate="0"/>
+  <xacro:joint_module_diff_drive parent="${name}" prefix="${prefix}" instance="1" scale="${scale}" rotate="0"/>
   <xacro:sm_wheel parent="${prefix}_jm_link_1" prefix="${prefix}" instance="1" dia="${JMwidth+0.3}" length="0.2" rotate="1" x="-1" y="0"/>
   <xacro:sm_wheel parent="${prefix}_jm_link_2" prefix="${prefix}" instance="2" dia="${JMwidth+0.3}" length="0.2" rotate="1" x="1" y="0"/>
@@ -43,9 +38,7 @@
   <xacro:initialising_frame name="base_footprint" child="1_jm_link2_0" scale="1" prefix="1"/>
   <gazebo>
-<!--
     <plugin name="gazebo_ros_control" filename="libgazebo_ros_control.so">
       <robotNamespace>/mrs</robotNamespace>
     </plugin>
--->
   </gazebo>
 </robot>

File: mrs_description/robots/JM2W2.xacro (robot description, xacro)
@@ -9,11 +9,6 @@
   <xacro:include filename="$(find mrs_description)/urdf/materials.urdf.xacro" />
 -->
-  <xacro:macro name="initialising_frame" params="name child scale prefix">
+  <xacro:macro name="initialising_frame" params="name scale prefix">
   <link name="${name}">
-    <inertial>
-      <mass value="0.1"/>
-      <origin xyz="0 0 0" rpy="0 0 0"/>
-      <inertia ixx="1.0" ixy="0.0" ixz="0.0" iyy="1.0" iyz="0.0" izz="1.0"/>
-    </inertial>
     <visual>
       <origin xyz="0 0 0" rpy="0 0 0"/>
@@ -35,17 +30,18 @@
   </joint>
   <link name="${name}_dummy"/>
-  <xacro:pcm_module parent="${name}" prefix="${prefix}" instance="1" scale="${scale}" len="0.3" z="0.15" />
-  <xacro:joint_module parent="${name}" prefix="${prefix}" instance="1" scale="${scale}" rotate="0"/>
-  <xacro:sm_wheel parent="${prefix}_jm_link_1" prefix="${prefix}" instance="1" dia="${JMwidth+0.3}" length="0.2" rotate="1" x="-1" y="0"/>
-  <xacro:sm_wheel parent="${prefix}_jm_link_2" prefix="${prefix}" instance="2" dia="${JMwidth+0.3}" length="0.2" rotate="1" x="1" y="0"/>
+  <xacro:pcm_module parent="${name}" prefix="${prefix}" instance="1" scale="${scale}" len="0.35" z="0" x="0.175" rotate="0" />
+  <xacro:pcm_module parent="${name}" prefix="${prefix}" instance="2" scale="${scale}" len="0.35" z="0" x="-0.175" rotate="2"/>
+  <xacro:joint_module_3DOF parent="${prefix}_pcm_link_1" prefix="1" instance="1" scale="${scale}" rotate="0"/>
+  <xacro:joint_module_3DOF parent="${prefix}_pcm_link_2" prefix="2" instance="1" scale="${scale}" rotate="0"/>
+  <xacro:sm_wheel parent="1_jm_link_2" prefix="${prefix}" instance="1" dia="${JMwidth+0.3}" length="0.2" rotate="1" x="1" y="0"/>
+  <xacro:sm_wheel parent="2_jm_link_2" prefix="${prefix}" instance="2" dia="${JMwidth+0.3}" length="0.2" rotate="1" x="1" y="0"/>
+  <xacro:diff_drive ljoint="2_jm_joint_2" rjoint="1_jm_joint_2" parent="${name}_dummy"  />
   </xacro:macro>
-<!-- For 1 Jm mobile robot -->
-  <xacro:initialising_frame name="base_footprint" child="1_jm_link2_0" scale="1" prefix="1"/>
+<!-- For 2 JM 2 PC 2 WM mobile robot -->
+  <xacro:initialising_frame name="base_footprint" scale="1" prefix="mrs"/>
   <gazebo>
-<!--
     <plugin name="gazebo_ros_control" filename="libgazebo_ros_control.so">
       <robotNamespace>/mrs</robotNamespace>
     </plugin>
--->
   </gazebo>
 </robot>

File: mrs_description/urdf/simplified_mrs.xacro (robot description, xacro)
@@ -1,6 +1,4 @@
 <?xml version="1.0"?>
 <robot name="mrs" xmlns:xacro="http://www.ros.org/wiki/xacro">
-  <!-- Constants for robot -->
-  <xacro:include filename="$(find mrs_description)/urdf/common_mrs.xacro" />
   <!-- Import Rviz colors -->
   <xacro:include filename="$(find mrs_description)/urdf/materials.urdf.xacro" />
@@ -8,13 +6,21 @@
   <xacro:property name="JMwidth" value=".4" />
   <xacro:property name="JMheight" value=".3" />
-  <xacro:macro name="joint_module" params="parent prefix instance scale rotate">
-<!--
-Mobile robot with 2 or More JM
--->
-<!--
-    <xacro:jm_rec_link parent="${parent}" prefix="${prefix}" instance="${instance-1}" scale="${scale}" rotate="0"/>
-    <xacro:jm_sphere_link parent="${prefix}_jm_link_${instance-1}" prefix="${prefix}" instance="${instance}" scale="${scale}" type="revolute"/>
-    <xacro:jm_rec_link parent="${prefix}_jm_link2_${instance}" prefix="${prefix}" instance="${instance}" scale="${scale}" rotate="0" />
--->
+  <xacro:macro name="joint_module_diff_drive" params="parent prefix instance scale rotate">
+<!-- Mobile robot using 1 JM - joint 2 should be made fixed -->
+    <xacro:jm_sphere_link parent="${parent}" prefix="${prefix}" instance="0" scale="${scale}" type="fixed"/>
+    <xacro:jm_rec_link parent="${prefix}_jm_link2_0" prefix="${prefix}" instance="1" scale="${scale}" rotate="0" reflect="-1" translateX="0" translateY="0"/>
+    <xacro:jm_rec_link parent="${prefix}_jm_link2_0" prefix="${prefix}" instance="2" scale="${scale}" rotate="0" reflect="1" translateX="0" translateY="0"/>
+    <xacro:simple_transmission joint="${prefix}_jm_joint_1" />
+    <xacro:simple_transmission joint="${prefix}_jm_joint_2" />
+    <xacro:diff_drive ljoint="${prefix}_jm_joint_1" rjoint="${prefix}_jm_joint_2" parent="${parent}"  />
+  </xacro:macro>
+    <xacro:macro name="joint_module_3DOF_vertical" params="parent prefix instance scale rotate">
+<!-- Mobile robot with 2 or More JM  -->
+    <xacro:jm_rec_link parent="${parent}" prefix="${prefix}" instance="1" scale="${scale}" rotate="${rotate}" reflect="0" translateX="0" translateY="0.1"/>
+    <xacro:jm_sphere_link parent="${prefix}_jm_link_${instance}" prefix="${prefix}" instance="${instance}" scale="${scale}" type="revolute"/>
+    <xacro:jm_rec_link parent="${prefix}_jm_link2_${instance}" prefix="${prefix}" instance="2" scale="${scale}" rotate="0" reflect="1" translateX="0" translateY="0"/>
+    <xacro:simple_transmission joint="${prefix}_jm_joint_1" />
+    <xacro:simple_transmission joint="${prefix}_jm_joint_2" />
+    <xacro:simple_transmission joint="${prefix}_jm_joint2_1" />
 <!--
 Manipulator - rotate =1
@@ -25,20 +31,23 @@
     <xacro:jm_rec_link parent="${prefix}_jm_link2_${instance}" prefix="${prefix}" instance="${instance}" scale="${scale}" rotate="0" />
 -->
+  </xacro:macro>
+  <xacro:macro name="joint_module_3DOF" params="parent prefix instance scale rotate">
+<!-- Mobile robot with 2 or More JM  -->
+    <xacro:jm_rec_link parent="${parent}" prefix="${prefix}" instance="1" scale="${scale}" rotate="${rotate}" reflect="1" translateX="0" translateY="0"/>
+    <xacro:jm_sphere_link parent="${prefix}_jm_link_${instance}" prefix="${prefix}" instance="${instance}" scale="${scale}" type="revolute"/>
+    <xacro:jm_rec_link parent="${prefix}_jm_link2_${instance}" prefix="${prefix}" instance="2" scale="${scale}" rotate="0" reflect="1" translateX="0" translateY="0"/>
+    <xacro:simple_transmission joint="${prefix}_jm_joint_1" />
+    <xacro:simple_transmission joint="${prefix}_jm_joint_2" />
+    <xacro:simple_transmission joint="${prefix}_jm_joint2_1" />
 <!--
-Mobile robot using 1 JM - joint 2 should be made fixed
+Manipulator - rotate =1
 -->
-    <xacro:jm_sphere_link parent="${parent}" prefix="${prefix}" instance="${instance-1}" scale="${scale}" type="fixed"/>
-    <xacro:jm_rec_link parent="${prefix}_jm_link2_${instance-1}" prefix="${prefix}" instance="${instance-2}" scale="${scale}" rotate="0"/>
 <!--
-    <xacro:simple_transmission joint="${instance}_${prefix}_j1" />
--->
-    <xacro:jm_rec_link parent="${prefix}_jm_link2_${instance-1}" prefix="${prefix}" instance="${instance}" scale="${scale}" rotate="0" />
-    <xacro:sm_wheel parent="${prefix}_jm_link_${instance}" prefix="${prefix}" instance="${instance}" dia="${JMwidth+0.2}" length="0.1" rotate="1" x="1" />
-    <xacro:sm_wheel parent="${prefix}_jm_link_${instance-2}" prefix="${prefix}" instance="${instance-2}" dia="${JMwidth+0.2}" length="0.1" rotate="1" x="-1" />
-<!--
-    <xacro:diff_drive ljoint="${prefix}_jm_joint_${instance-2}" rjoint="${prefix}_jm_joint_${instance}" parent="${parent}"  />
+    <xacro:jm_rec_link parent="${parent}" prefix="${prefix}" instance="${instance-1}" scale="${scale}" rotate="1"/>
+    <xacro:jm_sphere_link parent="${prefix}_jm_link_${instance-1}" prefix="${prefix}" instance="${instance}" scale="${scale}" type="revolute" />
+    <xacro:jm_rec_link parent="${prefix}_jm_link2_${instance}" prefix="${prefix}" instance="${instance}" scale="${scale}" rotate="0" />
 -->
   </xacro:macro>
-  <xacro:macro name="jm_rec_link" params="parent prefix instance scale rotate">
+  <xacro:macro name="jm_rec_link" params="parent prefix instance scale rotate reflect translateX translateY">
     <link name="${prefix}_jm_link_${instance}">
       <visual>
@@ -49,5 +58,4 @@
         </material>
       </visual>
-<!--
       <collision>
         <geometry>
@@ -55,5 +63,4 @@
         </geometry>
       </collision>
--->
       <xacro:default_inertial mass="1" I_tensor="1"/>
     </link>
@@ -62,10 +69,7 @@
       <child link="${prefix}_jm_link_${instance}" />
       <axis xyz="1 0 0"/>
-      <origin xyz="${(instance)*(JMlen+JMwidth)/2} 0 0" rpy="0 ${-rotate*pi/2} 0" />
+      <origin xyz="${(reflect)*(JMlen+JMwidth)/2} ${translateX} ${translateY}" rpy="0 ${-rotate*pi/2} 0" />
     </joint>
-    <gazebo reference = "${prefix}_jm_link_${instance}">
-      <material>Gazebo/Grey</material>
-      <selfCollide>false</selfCollide>
-    </gazebo>
+      <xacro:gazebo_visual link="${prefix}_jm_link_${instance}" visual="Grey" />
   </xacro:macro>
     <xacro:macro name="jm_sphere_link" params="parent prefix instance scale type">
@@ -78,5 +82,4 @@
           </material>
         </visual>
-<!--
         <collision>
           <geometry>
@@ -84,5 +87,4 @@
           </geometry>
         </collision>
--->
         <xacro:default_inertial mass="1" I_tensor="1"/>
       </link>
@@ -95,10 +97,8 @@
         upper="${pi/2}" />
       </joint>
-      <gazebo reference = "${prefix}_jm_link2_${instance}">
-        <material>Gazebo/Grey</material>
-        <selfCollide>false</selfCollide>
-      </gazebo>
+      <xacro:gazebo_visual link="${prefix}_jm_link2_${instance}" visual="Grey" />
     </xacro:macro>
     <xacro:macro name="diff_drive" params="ljoint rjoint parent">
+      <!-- CONTROLLERS -->
       <gazebo>
         <plugin name="differential_drive_controller" filename="libgazebo_ros_diff_drive.so">
@@ -107,8 +107,8 @@
           <leftJoint>${ljoint}</leftJoint>
           <rightJoint>${rjoint}</rightJoint>
-          <wheelSeparation>0.5380</wheelSeparation>
-          <wheelDiameter>0.2410</wheelDiameter>
+          <wheelSeparation>0.6</wheelSeparation>
+          <wheelDiameter>0.6</wheelDiameter>
           <torque>20</torque>
-          <commandTopic>cmd_vel</commandTopic>
+          <commandTopic>mrs/cmd_vel</commandTopic>
           <odometryTopic>odom</odometryTopic>
           <odometryFrame>odom</odometryFrame>
@@ -117,5 +117,5 @@
     </gazebo>
     </xacro:macro>
-    <xacro:macro name="pcm_cube_link" params="parent prefix instance scale len">
+    <xacro:macro name="pcm_module" params="parent prefix instance scale len z x rotate">
       <link name="${prefix}_pcm_link_${instance}">
         <visual>
@@ -126,5 +126,4 @@
           </material>
         </visual>
-<!--
         <collision>
           <geometry>
@@ -132,12 +131,12 @@
           </geometry>
         </collision>
--->
-        <xacro:default_inertial mass="1" I_tensor="1"/>
+        <xacro:default_inertial mass="0.01" I_tensor="1"/>
       </link>
       <joint name="${prefix}_pcm_joint_${instance}" type="fixed">
         <parent link="${parent}" />
         <child link="${prefix}_pcm_link_${instance}" />
-        <origin xyz="0 0 0.55" rpy="0 0 0" />
+        <origin xyz="${x} 0 ${z}" rpy="0 ${-rotate*pi/2} 0" />
       </joint>
+      <xacro:gazebo_visual link="${prefix}_pcm_link_${instance}" visual="Blue" />
     </xacro:macro>
   <xacro:macro name="cuboid_inertial" params="mass len height width">
@@ -157,5 +156,5 @@
     </inertial>
   </xacro:macro>
-  <xacro:macro name="sm_wheel" params="parent prefix instance dia length rotate x ">
+  <xacro:macro name="sm_wheel" params="parent prefix instance dia length rotate x y">
     <link name="${prefix}_sm_wheel_link_${instance}">
       <visual>
@@ -176,10 +175,24 @@
       <parent link="${parent}" />
       <child link="${prefix}_sm_wheel_link_${instance}" />
-      <origin xyz="${x*((JMlen+length)/2)} 0 0" rpy=" 0 ${rotate*pi/2} 0" />
+      <origin xyz="${x*((JMlen+length)/2)} ${y} 0" rpy=" 0 ${rotate*pi/2} 0" />
     </joint>
-    <gazebo reference = "${prefix}_sm_wheel_link_${instance}">
-      <material>Gazebo/Orange</material>
+    <xacro:gazebo_visual link="${prefix}_sm_wheel_link_${instance}" visual="White" />
+  </xacro:macro>
+  <xacro:macro name="gazebo_visual" params="link visual">
+    <gazebo reference = "${link}">
+      <material>Gazebo/${visual}</material>
       <selfCollide>false</selfCollide>
     </gazebo>
   </xacro:macro>
+    <!-- Transmission's Macro -->
+  <macro name="simple_transmission" params="joint">
+    <transmission name="${joint}tran">
+      <type>transmission_interface/SimpleTransmission</type>
+      <joint name="${joint}" />
+      <actuator name="${joint}_motor">
+        <hardwareInterface>EffortJointInterface</hardwareInterface>
+        <mechanicalReduction>1</mechanicalReduction>
+      </actuator>
+    </transmission>
+  </macro>
 </robot>
