Commit message: For Hotcell tests - fusion facility evaluation

File: mrs_description/robots/A2M_prismatic.xacro (robot description, xacro)
@@ -1,88 +1,90 @@
 <?xml version="1.0"?>
 <robot name="mrs" xmlns:xacro="http://www.ros.org/wiki/xacro">
-	<!-- Constants for robot -->
-	<xacro:include filename="$(find mrs_description)/urdf/common_mrs.xacro" />
-	<!-- Import all Gazebo-customization elements, including Gazebo colors -->
-	<xacro:include filename="$(find mrs_description)/urdf/JM/jm.xacro" />
-	<xacro:include filename="$(find mrs_description)/urdf/PCM/pcm.xacro" />
-	<xacro:include filename="$(find mrs_description)/urdf/power_base/sm_other.urdf.xacro" />
-	<!-- Used for fixing robot to Gazebo 'base_link' -->
-	<link name="world" />
-	<!-- Working copy -->
+    <!-- Constants for robot -->
+    <xacro:include filename="$(find mrs_description)/urdf/common_mrs.xacro" />
+    <!-- Import all Gazebo-customization elements, including Gazebo colors -->
+    <xacro:include filename="$(find mrs_description)/urdf/JM/jm.xacro" />
+    <xacro:include filename="$(find mrs_description)/urdf/PCM/pcm.xacro" />
+    <xacro:include filename="$(find mrs_description)/urdf/power_base/sm_other.urdf.xacro" />
+    <!-- Used for fixing robot to Gazebo 'base_link' -->
+    <link name="world" />
+    <!-- Working copy -->
 <!--
-	<joint name="fixed" type="fixed">
-		<origin xyz="0 0 0.01" rpy="0 0 0" />
-		<parent link="world" />
-		<child link="base_footprint" />
-	</joint>
+    <joint name="fixed" type="fixed">
+        <origin xyz="0 0 0.01" rpy="0 0 0" />
+        <parent link="world" />
+        <child link="base_footprint" />
+    </joint>
 -->
-	<!-- Fictitious Base Link is a fictitious link(frame) that is on the ground below
-		base_link origin, -->
-	<!-- Base Link -->
+    <!-- Fictitious Base Link is a fictitious link(frame) that is on the ground below
+        base_link origin, -->
+    <!-- Base Link -->
 <!--
-	<link name="base_footprint">
-		<inertial>
-			<mass value="1.0" />
-			<origin xyz="0 0 0" />
-			<inertia ixx="0.01" ixy="0.0" ixz="0.0" iyy="0.01" iyz="0.0"
-				izz="0.01" />
-		</inertial>
-		<visual>
-			<origin xyz="0 0 0" rpy="0 0 0" />
-			<geometry>
-				<box size="0.01 0.01 0.01" />
-			</geometry>
-		</visual>
-		<collision>
-			<origin xyz="0 0 0.01" rpy="0 0 0" />
-			<geometry>
-				<box size="0.001 0.001 0.001" />
-			</geometry>
-		</collision>
-	</link>
+    <link name="base_footprint">
+        <inertial>
+            <mass value="1.0" />
+            <origin xyz="0 0 0" />
+            <inertia ixx="0.01" ixy="0.0" ixz="0.0" iyy="0.01" iyz="0.0"
+                izz="0.01" />
+        </inertial>
+        <visual>
+            <origin xyz="0 0 0" rpy="0 0 0" />
+            <geometry>
+                <box size="0.01 0.01 0.01" />
+            </geometry>
+        </visual>
+        <collision>
+            <origin xyz="0 0 0.01" rpy="0 0 0" />
+            <geometry>
+                <box size="0.001 0.001 0.001" />
+            </geometry>
+        </collision>
+    </link>
 -->
-	<!-- Initial the xacros calls -->
+    <!-- Initial the xacros calls -->
+    <xacro:JM1 name="JM" prefix="L1" instance="1"  parent="world" />
+    <xacro:PcModule parent="L1_PCmodule" prefix="L2" instance="2" />
+    <xacro:PcModule parent="1_L1_j2_link" prefix="L1" instance="1" />
+    <xacro:PcModule_Prismatic_arm parent="L1_PCmodule" prefix="L2_prismatic" reflect="1" shift="0.07"/>
+    <xacro:JM2 name="JM1" prefix="L1" instance="2"  parent="L2_prismatic_PCmodule" reflect="1" shift="0.035" shift2="0"/>
+    <xacro:SMRadprobe parent="2_L1_w1_link" prefix="L1" reflect="0" instance="1" />
+<!-- To remove fixed links between the arm links new robot configuration -->
 <!--
-	<xacro:JM1 name="JM" prefix="L1" instance="1"  parent="base_footprint" />
-	<xacro:PcModule parent="L1_PCmodule" prefix="L2" instance="2" />
-	<xacro:PcModule parent="1_L1_j2_link" prefix="L1" instance="1" />
-	<xacro:PcModule_Prismatic_arm parent="L1_PCmodule" prefix="L2_prismatic" reflect="1" shift="0.07"/>
-	<xacro:JM2 name="JM1" prefix="L1" instance="2"  parent="L2_prismatic_PCmodule" reflect="1" shift="0.035" shift2="0"/>
-	<xacro:SMRadprobe parent="2_L1_w1_link" prefix="L1" reflect="0" instance="1" />
+    <xacro:JM1_kinematic name="JM" prefix="L1" instance="1"  parent="world" />
+    <xacro:PcModule_Prismatic_kinematic parent="1_L1_j2_link" prefix="L1_prismatic" reflect="1" shift="0.07"/>
+    <xacro:JM2_kinematic name="JM1" prefix="L1" instance="2"  parent="L1_prismatic_PCmodule" reflect="0" shift="0.125" shift2="0"/>
 -->
-<!-- To remove fixed links between the arm links new robot configuration -->
-	<xacro:JM1_kinematic name="JM" prefix="L1" instance="1"  parent="world" />
 <!--
-	<xacro:PcModule_Prismatic_kinematic parent="1_L1_j2_link" prefix="L1_prismatic" reflect="1" shift="0.07"/>
-	<xacro:JM2_kinematic name="JM1" prefix="L1" instance="2"  parent="L1_prismatic_PCmodule" reflect="0" shift="0.125" shift2="0"/>
+    <xacro:JM2_kinematic name="JM1" prefix="L1" instance="2"  parent="1_L1_j2_link" reflect="0" shift="0.125" shift2="0"/>
 -->
-	<xacro:JM2_kinematic name="JM1" prefix="L1" instance="2"  parent="1_L1_j2_link" reflect="0" shift="0.125" shift2="0"/>
-		<joint name="1_L1_SMprobe_joint" type="fixed">
-			<parent link="2_L1_j3_link" />
-			<child link="1_L1_rad_pole" />
-			<origin rpy="${pi/2} 0 0" xyz="0 0.07 0" />
-		</joint>
-		<link name="1_L1_rad_pole">
-			<visual>
-				<geometry>
-					<cylinder length="0.1" radius=".01" />
-				</geometry>
-				<origin rpy="0 0 0 " xyz="0 0 0" />
-				<material name="Gray">
-					<color rgba=".7 .7 .7 1" />
-				</material>
-			</visual>
-			<collision>
-				<geometry>
-					<cylinder length="0.06" radius=".01" />
-				</geometry>
-			</collision>
-		</link>
-	<!-- ros_control plugin -->
-	<gazebo>
-		<plugin name="mrs_ros_control" filename="libgazebo_ros_control.so">
-			<controlPeriod>0.001</controlPeriod>
-			<robotNamespace>/mrs</robotNamespace>
-		</plugin>
-	</gazebo>
+<!--
+        <joint name="1_L1_SMprobe_joint" type="fixed">
+            <parent link="2_L1_j3_link" />
+            <child link="1_L1_rad_pole" />
+            <origin rpy="${pi/2} 0 0" xyz="0 0.07 0" />
+        </joint>
+        <link name="1_L1_rad_pole">
+            <visual>
+                <geometry>
+                    <cylinder length="0.1" radius=".01" />
+                </geometry>
+                <origin rpy="0 0 0 " xyz="0 0 0" />
+                <material name="Gray">
+                    <color rgba=".7 .7 .7 1" />
+                </material>
+            </visual>
+            <collision>
+                <geometry>
+                    <cylinder length="0.06" radius=".01" />
+                </geometry>
+            </collision>
+        </link>
+-->
+    <!-- ros_control plugin -->
+    <gazebo>
+        <plugin name="mrs_ros_control" filename="libgazebo_ros_control.so">
+            <controlPeriod>0.001</controlPeriod>
+            <robotNamespace>/mrs</robotNamespace>
+        </plugin>
+    </gazebo>
 </robot>

File: mrs_description/urdf/PCM/pcm.xacro (robot description, xacro)
@@ -1,150 +1,174 @@
 <?xml version="1.0"?>
 <robot name="mrs" xmlns:xacro="http://www.ros.org/wiki/xacro">
-	<!-- Constants for robot -->
-	<xacro:include filename="$(find mrs_description)/urdf/common_mrs.xacro" />
-	<!-- Import all Gazebo-customization elements, including Gazebo colors -->
-	<xacro:include filename="$(find mrs_description)/urdf/PCM/pcm.gazebo.xacro" />
-	<!-- Import Rviz colors -->
-	<xacro:include filename="$(find mrs_description)/urdf/materials.xacro" />
-	<xacro:macro name="default_inertial" params="mass I_tensor">
-		<inertial>
-			<mass value="${mass}" />
+    <!-- Constants for robot -->
+    <xacro:include filename="$(find mrs_description)/urdf/common_mrs.xacro" />
+    <!-- Import all Gazebo-customization elements, including Gazebo colors -->
+    <xacro:include filename="$(find mrs_description)/urdf/PCM/pcm.gazebo.xacro" />
+    <!-- Import Rviz colors -->
+    <xacro:include filename="$(find mrs_description)/urdf/materials.xacro" />
+    <xacro:macro name="default_inertial" params="mass I_tensor">
+        <inertial>
+            <mass value="${mass}" />
 <!--
-			Inertia of a cuboid - ml2/6
+            Inertia of a cuboid - ml2/6
 -->
-			<inertia ixx="${I_tensor*1.0}" ixy="0.0" ixz="0.0" iyy="${I_tensor*1.0}" iyz="0.0"
-				izz="${I_tensor*1.0}" />
-		</inertial>
-	</xacro:macro>
-	<xacro:macro name="PcModule" params="parent prefix instance">
-		<link name="${prefix}_PCmodule">
-			<visual>
-				<geometry>
-					<box size="0.07 0.07 0.07" />
-				</geometry>
-				<material name="Blue">
-				</material>
-			</visual>
-			<collision>
-				<geometry>
-					<box size="0.07 0.07 0.04" />
-				</geometry>
-			</collision>
-			<xacro:default_inertial mass="0.15" I_tensor="8.166e-4"/>
-		</link>
-		<joint name="${instance}_${prefix}_mbase_jointW1" type="fixed">
-			<origin xyz="0 0 ${instance*0.035}" rpy="0 0 0" />
-			<child link="${prefix}_PCmodule" />
-			<parent link="${parent}" />
-		</joint>
-	<!-- Gazebo  -->
-	<xacro:PCMG name="${prefix}_pcm_gazebo" prefix="${prefix}" instance="${instance}" />
-	</xacro:macro>
-	<xacro:macro name="PcModule_Prismatic" params="parent prefix reflect">
-		<link name="${prefix}_PCmodule">
-			<visual>
-				<geometry>
-					<box size="0.07 0.05 0.05" />
-				</geometry>
-				<material name="Orange">
-				</material>
-			</visual>
-			<xacro:default_inertial mass="0.15" I_tensor="8.166e-4"/>
-		</link>
-		<joint name="${prefix}_mbase_jointW1" type="prismatic">
-			<origin xyz="0 0 ${reflect*0.035}" rpy="0 ${-reflect*pi/2} 0" />
-			<child link="${prefix}_PCmodule" />
-			<parent link="${parent}" />
-			<limit lower="0" upper="0.03" effort="${max_effort}"
-			velocity="${max_velocity}" />
-		</joint>
-	<simple_transmission joint="${prefix}_mbase_jointW1" />
-	<!-- Gazebo  -->
-	<xacro:PCMG name="${prefix}_pcm_gazebo" prefix="${prefix}" instance="${reflect}" />
-	</xacro:macro>
-	<xacro:macro name="PcModule_Prismatic_arm" params="parent prefix reflect shift">
-		<link name="${prefix}_PCmodule">
-			<visual>
-				<geometry>
-					<box size="0.07 0.05 0.05" />
-				</geometry>
-				<material name="Orange">
-				</material>
-			</visual>
-			<xacro:default_inertial mass="0.15" I_tensor="8.166e-4"/>
-		</link>
-		<joint name="${prefix}_mbase_jointW1" type="prismatic">
-			<origin xyz="0 0 ${reflect*shift}" rpy="0 ${-reflect*pi/2} 0" />
-			<child link="${prefix}_PCmodule" />
-			<parent link="${parent}" />
-			<limit lower="0" upper="0.07" effort="${max_effort}"
-			velocity="${max_velocity}" />
-		</joint>
-	<simple_transmission joint="${prefix}_mbase_jointW1" />
-	<!-- Gazebo  -->
-	<xacro:PCMG name="${prefix}_pcm_gazebo" prefix="${prefix}" instance="${reflect}" />
-	</xacro:macro>
-	<xacro:macro name="PcModule_Prismatic" params="parent prefix reflect">
-		<link name="${prefix}_PCmodule">
-			<visual>
-				<geometry>
-					<box size="0.07 0.05 0.05" />
-				</geometry>
-				<material name="Orange">
-				</material>
-			</visual>
-			<xacro:default_inertial mass="0.15" I_tensor="8.166e-4"/>
-		</link>
-		<joint name="${prefix}_mbase_jointW1" type="prismatic">
-			<origin xyz="0 0 ${reflect*0.035}" rpy="0 ${-reflect*pi/2} 0" />
-			<child link="${prefix}_PCmodule" />
-			<parent link="${parent}" />
-			<limit lower="0" upper="0.03" effort="${max_effort}"
-			velocity="${max_velocity}" />
-		</joint>
-	<simple_transmission joint="${prefix}_mbase_jointW1" />
-	<!-- Gazebo  -->
-	<xacro:PCMG name="${prefix}_pcm_gazebo" prefix="${prefix}" instance="${reflect}" />
-	</xacro:macro>
-	<xacro:macro name="PcModule_Prismatic_kinematic" params="parent prefix reflect shift">
-		<link name="${prefix}_PCmodule">
-			<visual>
-				<geometry>
-					<box size="0.14 0.06 0.05" />
-				</geometry>
-				<material name="Blue">
-				</material>
-			</visual>
-			<xacro:default_inertial mass="0.15" I_tensor="8.166e-4"/>
-		</link>
-		<joint name="${prefix}_mbase_jointW1" type="prismatic">
-			<origin xyz="0 0 ${reflect*shift}" rpy="0 ${-reflect*pi/2} 0" />
-			<child link="${prefix}_PCmodule" />
-			<parent link="${parent}" />
-			<limit lower="0" upper="0.07" effort="${max_effort}"
-			velocity="${max_velocity}" />
-		</joint>
-	<simple_transmission joint="${prefix}_mbase_jointW1" />
-	<!-- Gazebo  -->
-	<xacro:PCMG name="${prefix}_pcm_gazebo" prefix="${prefix}" instance="${reflect}" />
-	</xacro:macro>
-	<xacro:macro name="PcModule_solid" params="parent prefix reflect">
-		<link name="${prefix}_PCmodule">
-			<visual>
-				<geometry>
-					<box size="0.07 0.05 0.05" />
-				</geometry>
-				<material name="Orange">
-				</material>
-			</visual>
-			<xacro:default_inertial mass="0.15" I_tensor="8.166e-4"/>
-		</link>
-		<joint name="${prefix}_mbase_jointW1" type="fixed">
-			<origin xyz="0 0 ${reflect*0.035}" rpy="0 ${-reflect*pi/2} 0" />
-			<child link="${prefix}_PCmodule" />
-			<parent link="${parent}" />>
-		</joint>
-	<!-- Gazebo  -->
-	<xacro:PCMG name="${prefix}_pcm_gazebo" prefix="${prefix}" instance="${reflect}" />
-	</xacro:macro>
+            <inertia ixx="${I_tensor*1.0}" ixy="0.0" ixz="0.0" iyy="${I_tensor*1.0}" iyz="0.0"
+                izz="${I_tensor*1.0}" />
+        </inertial>
+    </xacro:macro>
+    <xacro:macro name="PcModule_flex" params="parent prefix instance shift">
+        <link name="${prefix}_PCmodule">
+            <visual>
+                <geometry>
+                    <box size="0.07 0.07 0.07" />
+                </geometry>
+                <material name="Blue">
+                </material>
+            </visual>
+            <collision>
+                <geometry>
+                    <box size="0.07 0.07 0.04" />
+                </geometry>
+            </collision>
+            <xacro:default_inertial mass="0.15" I_tensor="8.166e-4"/>
+        </link>
+        <joint name="${instance}_${prefix}_mbase_jointW1" type="fixed">
+            <origin xyz="0 ${shift*instance*0.035} 0" rpy=" ${-pi/2} 0 0" />
+            <child link="${prefix}_PCmodule" />
+            <parent link="${parent}" />
+        </joint>
+    <!-- Gazebo  -->
+    <xacro:PCMG name="${prefix}_pcm_gazebo" prefix="${prefix}" instance="${instance}" />
+    </xacro:macro>
+    <xacro:macro name="PcModule" params="parent prefix instance">
+        <link name="${prefix}_PCmodule">
+            <visual>
+                <geometry>
+                    <box size="0.07 0.07 0.07" />
+                </geometry>
+                <material name="Blue">
+                </material>
+            </visual>
+            <collision>
+                <geometry>
+                    <box size="0.07 0.07 0.04" />
+                </geometry>
+            </collision>
+            <xacro:default_inertial mass="0.15" I_tensor="8.166e-4"/>
+        </link>
+        <joint name="${instance}_${prefix}_mbase_jointW1" type="fixed">
+            <origin xyz="0 0 ${instance*0.035}" rpy="0 0 0" />
+            <child link="${prefix}_PCmodule" />
+            <parent link="${parent}" />
+        </joint>
+    <!-- Gazebo  -->
+    <xacro:PCMG name="${prefix}_pcm_gazebo" prefix="${prefix}" instance="${instance}" />
+    </xacro:macro>
+    <xacro:macro name="PcModule_Prismatic" params="parent prefix reflect">
+        <link name="${prefix}_PCmodule">
+            <visual>
+                <geometry>
+                    <box size="0.07 0.05 0.05" />
+                </geometry>
+                <material name="Orange">
+                </material>
+            </visual>
+            <xacro:default_inertial mass="0.15" I_tensor="8.166e-4"/>
+        </link>
+        <joint name="${prefix}_mbase_jointW1" type="prismatic">
+            <origin xyz="0 0 ${reflect*0.035}" rpy="0 ${-reflect*pi/2} 0" />
+            <child link="${prefix}_PCmodule" />
+            <parent link="${parent}" />
+            <limit lower="0" upper="0.03" effort="${max_effort}"
+            velocity="${max_velocity}" />
+        </joint>
+    <simple_transmission joint="${prefix}_mbase_jointW1" />
+    <!-- Gazebo  -->
+    <xacro:PCMG name="${prefix}_pcm_gazebo" prefix="${prefix}" instance="${reflect}" />
+    </xacro:macro>
+    <xacro:macro name="PcModule_Prismatic_arm" params="parent prefix reflect shift">
+        <link name="${prefix}_PCmodule">
+            <visual>
+                <geometry>
+                    <box size="0.07 0.05 0.05" />
+                </geometry>
+                <material name="Orange">
+                </material>
+            </visual>
+            <xacro:default_inertial mass="0.15" I_tensor="8.166e-4"/>
+        </link>
+        <joint name="${prefix}_mbase_jointW1" type="prismatic">
+            <origin xyz="0 0 ${reflect*shift}" rpy="0 ${-reflect*pi/2} 0" />
+            <child link="${prefix}_PCmodule" />
+            <parent link="${parent}" />
+            <limit lower="0" upper="0.07" effort="${max_effort}"
+            velocity="${max_velocity}" />
+        </joint>
+    <simple_transmission joint="${prefix}_mbase_jointW1" />
+    <!-- Gazebo  -->
+    <xacro:PCMG name="${prefix}_pcm_gazebo" prefix="${prefix}" instance="${reflect}" />
+    </xacro:macro>
+    <xacro:macro name="PcModule_Prismatic" params="parent prefix reflect">
+        <link name="${prefix}_PCmodule">
+            <visual>
+                <geometry>
+                    <box size="0.07 0.05 0.05" />
+                </geometry>
+                <material name="Orange">
+                </material>
+            </visual>
+            <xacro:default_inertial mass="0.15" I_tensor="8.166e-4"/>
+        </link>
+        <joint name="${prefix}_mbase_jointW1" type="prismatic">
+            <origin xyz="0 0 ${reflect*0.035}" rpy="0 ${-reflect*pi/2} 0" />
+            <child link="${prefix}_PCmodule" />
+            <parent link="${parent}" />
+            <limit lower="0" upper="0.03" effort="${max_effort}"
+            velocity="${max_velocity}" />
+        </joint>
+    <simple_transmission joint="${prefix}_mbase_jointW1" />
+    <!-- Gazebo  -->
+    <xacro:PCMG name="${prefix}_pcm_gazebo" prefix="${prefix}" instance="${reflect}" />
+    </xacro:macro>
+    <xacro:macro name="PcModule_Prismatic_kinematic" params="parent prefix reflect shift">
+        <link name="${prefix}_PCmodule">
+            <visual>
+                <geometry>
+                    <box size="0.14 0.06 0.05" />
+                </geometry>
+                <material name="Blue">
+                </material>
+            </visual>
+            <xacro:default_inertial mass="0.15" I_tensor="8.166e-4"/>
+        </link>
+        <joint name="${prefix}_mbase_jointW1" type="prismatic">
+            <origin xyz="0 0 ${reflect*shift}" rpy="0 ${-reflect*pi/2} 0" />
+            <child link="${prefix}_PCmodule" />
+            <parent link="${parent}" />
+            <limit lower="0" upper="0.07" effort="${max_effort}"
+            velocity="${max_velocity}" />
+        </joint>
+    <simple_transmission joint="${prefix}_mbase_jointW1" />
+    <!-- Gazebo  -->
+    <xacro:PCMG name="${prefix}_pcm_gazebo" prefix="${prefix}" instance="${reflect}" />
+    </xacro:macro>
+    <xacro:macro name="PcModule_solid" params="parent prefix reflect">
+        <link name="${prefix}_PCmodule">
+            <visual>
+                <geometry>
+                    <box size="0.07 0.05 0.05" />
+                </geometry>
+                <material name="Orange">
+                </material>
+            </visual>
+            <xacro:default_inertial mass="0.15" I_tensor="8.166e-4"/>
+        </link>
+        <joint name="${prefix}_mbase_jointW1" type="fixed">
+            <origin xyz="0 0 ${reflect*0.035}" rpy="0 ${-reflect*pi/2} 0" />
+            <child link="${prefix}_PCmodule" />
+            <parent link="${parent}" />>
+        </joint>
+    <!-- Gazebo  -->
+    <xacro:PCMG name="${prefix}_pcm_gazebo" prefix="${prefix}" instance="${reflect}" />
+    </xacro:macro>
 </robot>
