Commit message: backup

File: mrs_description/robots/2W1JM.xacro (robot description, xacro)
@@ -4,5 +4,5 @@
   <xacro:include filename="$(find mrs_description)/urdf/common_mrs.xacro" />
   <!-- Import all Gazebo-customization elements, including Gazebo colors -->
-  <xacro:include filename="$(find mrs_description)/urdf/JM/simplified_jm.xacro" />
+  <xacro:include filename="$(find mrs_description)/urdf/simplified_mrs.xacro" />
   <!-- materials for visualization -->
 <!--
@@ -30,19 +30,18 @@
   </link>
   <joint name="${name}_joint" type="fixed">
-    <origin xyz="0 0 0.5" rpy="0 0 0"/>
+    <origin xyz="0 0 0.2" rpy="0 0 0"/>
     <child link="${child}"/>
     <parent link="${name}"/>
   </joint>
-  <xacro:pcm_cube_link parent="${name}" prefix="${prefix}" instance="1" scale="${scale}" len="0.3" />
-  <xacro:joint_module parent="${child}" prefix="${prefix}" instance="1" scale="${scale}" />
+  <xacro:pcm_cube_link parent="${name}" prefix="${prefix}" instance="1" scale="${scale}" len="0.35" />
+  <xacro:joint_module parent="${name}" prefix="${prefix}" instance="1" scale="${scale}" rotate="0"/>
   </xacro:macro>
-  <xacro:initialising_frame name="base_footprint" child="1_pcm_link_1" scale="1" prefix="1"/>
+<!-- For 1 Jm mobile robot -->
+  <xacro:initialising_frame name="base_footprint" child="1_jm_link2_0.0" scale="1" prefix="1"/>
+<!-- For 2 Jm mobile robot -->
 <!--
-  <xacro:Ball_bearing mass="0.1" instance="1" dia="0.01" x="-0.045" y="0.0" z="-0.2" parent="base_footprint"/>
-  <xacro:Ball_bearing mass="0.1" instance="2" dia="0.01" x="-0.045" y="0.0" z="0.2" parent="base_footprint"/>
+ <xacro:initialising_frame name="base_footprint" child="1_jm_link_0.0" scale="1" prefix="1"/>
 -->
 <!--
-  <xacro:Ball_bearing mass="0.1" instance="1" dia="0.01" x="-0.055" y="0" z="-0.07" parent="base_footprint"/>
-  <xacro:Ball_bearing mass="0.1" instance="2" dia="0.01" x="-0.055" y="0" z="0.07" parent="base_footprint"/>
   <gazebo>
     <plugin name="gazebo_ros_controller_manager" filename="libgazebo_ros_control.so">
