Commit message: Commit for the fusion des eng

File: mrs_description/robots/2W1JM.xacro (robot description, xacro)
@@ -35,5 +35,5 @@
   </joint>
   <link name="${name}_dummy"/>
-  <xacro:pcm_module parent="${name}" prefix="${prefix}" instance="1" scale="${scale}" len="0.3" z="0.15" />
+  <xacro:pcm_module parent="${name}" prefix="${prefix}" instance="1" scale="${scale}" len="0.3" z="0.15" x="0" rotate="0"/>
   <xacro:joint_module parent="${name}" prefix="${prefix}" instance="1" scale="${scale}" rotate="0"/>
   <xacro:sm_wheel parent="${prefix}_jm_link_1" prefix="${prefix}" instance="1" dia="${JMwidth+0.3}" length="0.2" rotate="1" x="-1" y="0"/>

File: mrs_description/robots/A2M.xacro (robot description, xacro)
@@ -1,55 +1,61 @@
 <?xml version="1.0"?>
 <robot name="mrs" xmlns:xacro="http://www.ros.org/wiki/xacro">
-	<!-- Constants for robot -->
-	<xacro:include filename="$(find mrs_description)/urdf/common_mrs.xacro" />
-	<!-- Import all Gazebo-customization elements, including Gazebo colors -->
-	<xacro:include filename="$(find mrs_description)/urdf/JM/jm.xacro" />
-	<xacro:include filename="$(find mrs_description)/urdf/PCM/pcm.xacro" />
-	<!-- Used for fixing robot to Gazebo 'base_link' -->
-	<link name="world" />
-	<joint name="fixed" type="fixed">
-		<origin xyz="0 0 0.01" rpy="0 0 0" />
-		<parent link="world" />
-		<child link="base_footprint" />
-	</joint>
-	<!-- Fictitious Base Link is a fictitious link(frame) that is on the ground below
-		base_link origin, -->
-	<!-- Base Link -->
-	<link name="base_footprint">
-		<inertial>
-			<mass value="1.0" />
-			<origin xyz="0 0 0" />
-			<inertia ixx="0.01" ixy="0.0" ixz="0.0" iyy="0.01" iyz="0.0"
-				izz="0.01" />
-		</inertial>
-		<visual>
-			<origin xyz="0 0 0" rpy="0 0 0" />
-			<geometry>
-				<box size="0.01 0.01 0.01" />
-			</geometry>
-		</visual>
-		<collision>
-			<origin xyz="0 0 0.01" rpy="0 0 0" />
-			<geometry>
-				<box size="0.001 0.001 0.001" />
-			</geometry>
-		</collision>
-	</link>
-	<xacro:JM1 name="JM" prefix="L1" instance="1"  parent="base_footprint" />
-	<xacro:PcModule parent="1_L1_j2_link" prefix="L1" instance="1" />
-	<xacro:PcModule parent="L1_PCmodule" prefix="L2" instance="2" />
-	<xacro:JM2 name="JM1" prefix="L1" instance="2"  parent="L2_PCmodule" reflect="0" shift="0.035" shift2="1"/>
-	<!-- ros_control plugin -->
-	<gazebo>
-		<plugin name="mrs_ros_control" filename="libgazebo_ros_control.so">
-			<controlPeriod>0.001</controlPeriod>
-			<robotNamespace>/mrs</robotNamespace>
-		</plugin>
-	</gazebo>
+    <!-- Constants for robot -->
+    <xacro:include filename="$(find mrs_description)/urdf/common_mrs.xacro" />
+    <!-- Import all Gazebo-customization elements, including Gazebo colors -->
+    <xacro:include filename="$(find mrs_description)/urdf/JM/jm.xacro" />
+    <xacro:include filename="$(find mrs_description)/urdf/PCM/pcm.xacro" />
+    <!-- Used for fixing robot to Gazebo 'base_link' -->
+    <link name="world" />
+    <joint name="fixed" type="fixed">
+        <origin xyz="0 0 0.01" rpy="0 0 0" />
+        <parent link="world" />
+        <child link="base_footprint" />
+    </joint>
+    <!-- Fictitious Base Link is a fictitious link(frame) that is on the ground below
+        base_link origin, -->
+    <!-- Base Link -->
+    <link name="base_footprint">
+        <inertial>
+            <mass value="1.0" />
+            <origin xyz="0 0 0" />
+            <inertia ixx="0.01" ixy="0.0" ixz="0.0" iyy="0.01" iyz="0.0"
+                izz="0.01" />
+        </inertial>
+        <visual>
+            <origin xyz="0 0 0" rpy="0 0 0" />
+            <geometry>
+                <box size="0.01 0.01 0.01" />
+            </geometry>
+        </visual>
+        <collision>
+            <origin xyz="0 0 0.01" rpy="0 0 0" />
+            <geometry>
+                <box size="0.001 0.001 0.001" />
+            </geometry>
+        </collision>
+    </link>
 <!--
-	<xacro:JM1 name="JM" prefix="L1" instance="1"  parent="base_footprint"/>
-	<xacro:PcModule parent="1_L1_j2_link" prefix="L1" instance="1" />
-	<xacro:PcModule parent="L1_PCmodule" prefix="L2" instance="1" />
-	<xacro:JM2 name="JM1" prefix="L2" instance="2"  parent="L2_PCmodule"/>
+    <xacro:macro name="arm" params="parent prefix x y z instance">
+-->
+    <xacro:JM1 name="JM" prefix="L1" instance="1"  parent="base_footprint" />
+    <xacro:PcModule parent="1_L1_j2_link" prefix="L1" instance="1" />
+    <xacro:PcModule parent="L1_PCmodule" prefix="L12" instance="2" />
+    <xacro:JM2 name="JM1" prefix="L1" instance="2"  parent="L12_PCmodule" reflect="0" shift="0.035" shift2="1"/>
+<!--
+    </xacro:macro>
+-->
+    <!-- ros_control plugin -->
+    <gazebo>
+        <plugin name="mrs_ros_control" filename="libgazebo_ros_control.so">
+            <controlPeriod>0.001</controlPeriod>
+            <robotNamespace>/mrs</robotNamespace>
+        </plugin>
+    </gazebo>
+<!--
+    <xacro:JM1 name="JM" prefix="L1" instance="1"  parent="base_footprint"/>
+    <xacro:PcModule parent="1_L1_j2_link" prefix="L1" instance="1" />
+    <xacro:PcModule parent="L1_PCmodule" prefix="L2" instance="1" />
+    <xacro:JM2 name="JM1" prefix="L2" instance="2"  parent="L2_PCmodule"/>
 -->
 </robot>

File: mrs_description/robots/W2M_prismatic_type2.xacro (robot description, xacro)
@@ -5,4 +5,5 @@
     <!-- Import all Gazebo-customization elements, including Gazebo colors -->
     <xacro:include filename="$(find mrs_description)/urdf/power_base/ball_bearing.urdf.xacro" />
+    <xacro:include filename="$(find mrs_description)/urdf/power_base/sm_other.urdf.xacro" />
     <xacro:include filename="$(find mrs_description)/urdf/JM/jm.xacro" />
     <xacro:include filename="$(find mrs_description)/urdf/PCM/pcm.xacro" />
@@ -57,8 +58,10 @@
         <selfCollide>false</selfCollide>
     </gazebo>
-    <xacro:JM3_solid name="JM" prefix="W1" instance="1"  parent="W1_PCmodule" reflect="1" shift="0.035"/>
-    <xacro:PcModule_Prismatic parent="base_footprint" prefix="W1" reflect="-1" />
-    <xacro:PcModule_Prismatic parent="base_footprint" prefix="W2" reflect="1" />
-    <xacro:JM3_solid name="JM1" prefix="W1" instance="2"  parent="W2_PCmodule" reflect="-1" shift="0.035"/>
+  <xacro:PcModule_Prismatic parent="world" prefix="W3" reflect="3" />
+  <xacro:JM3_solid name="JM" prefix="W1" instance="1"  parent="W1_PCmodule" reflect="1" shift="0.035"/>
+  <xacro:PcModule_solid parent="base_footprint" prefix="W1" reflect="-1" />
+  <xacro:PcModule_solid parent="base_footprint" prefix="W2" reflect="1" />
+  <xacro:JM3_solid name="JM1" prefix="W1" instance="2"  parent="W2_PCmodule" reflect="-1" shift="0.035"/>
+  <xacro:SMRadprobe parent="W3_PCmodule" prefix="W4" reflect="0" instance="1" />
 <!--
     <xacro:Ball_bearing mass="0.1" instance="1" dia="0.05" x="-0.035" y="0" z="0.035" parent="base_footprint"/>

File: mrs_description/robots/power_base_pic2.xacro (robot description, xacro)
@@ -125,4 +125,5 @@
   </joint>
   <!-- inspection robot-->
+<!--
     <link name="robot2" />
 <joint name="fixed_robot2_joint" type="fixed">
@@ -134,5 +135,4 @@
         <axis xyz="1 0 0 " />
         <origin xyz="0 0 0.05" rpy="0 ${-pi/2} 0" />
-        <!-- <origin xyz="0 0 0.1" rpy="0 0 0" /> -->
         <parent link="robot2" />
         <child link="robot2_world_footprint" />
@@ -153,4 +153,5 @@
   <xacro:JM3 name="JM1" prefix="W1" instance="2"  parent="W2_PCmodule" reflect="-1" shift="0.035"/>
   <xacro:SMRadprobe parent="W3_PCmodule" prefix="W4" reflect="0" instance="1" />
+-->
   <!-- foot for arm-->
     <link name="robot1" >
@@ -173,13 +174,4 @@
 -->
 <!--
-    leg 1 - parent {instance}_${prefix}_camera_link
--->
-<!--
-    <xacro:JM1_armconnect name="JM" prefix="L1" instance="1"  parent="1_base_camera_link" />
-    <xacro:PcModule parent="1_L1_j2_link" prefix="L1" instance="1" />
-    <xacro:PcModule parent="L1_PCmodule" prefix="L12" instance="2" />
-    <xacro:JM2 name="JM1" prefix="L1" instance="2"  parent="L12_PCmodule" reflect="0" shift="0.035" shift2="1"/>
--->
-<!--
           Create the orientation joint
 -->
@@ -208,10 +200,5 @@
     <xacro:PcModule_Prismatic_arm parent="L22_PCmodule" prefix="L2_prismatic" reflect="1" shift="0.07"/>
     <xacro:JM2 name="JM1" prefix="L2" instance="2"  parent="L2_prismatic_PCmodule" reflect="1" shift="0.035" shift2="0"/>
-<!--
-    <xacro:SMRadprobe parent="2_L2_w1_link" prefix="L1" reflect="0" instance="1" />
--->
-<!--
-    <xacro:SMHand parent="2_L2_w1_link" prefix="L2" reflect="0" instance="1"/>
--->
+    <xacro:SMHand parent="2_L2_w1_link" prefix="L2" reflect="1" instance="1"/>
 <!--
 ARM 2
@@ -222,10 +209,10 @@
     <child link="arm2"/>
     <parent link="4_base_camera_link"/>
-     <limit lower="0" upper="-3" effort="${max_effort}"
+     <limit lower="${-pi}" upper="${pi}" effort="${max_effort}"
       velocity="${max_velocity}" />
   </joint>
   <link name="arm2_1" />
   <joint name="arm22_joint" type="revolute">
-    <origin xyz="0 0 0" rpy="0 0 ${-pi/2}"/>
+    <origin xyz="0 0 0" rpy="0 0 ${pi/2}"/>
     <child link="arm2_1"/>
     <parent link="arm2"/>
@@ -233,12 +220,54 @@
       velocity="${max_velocity}" />
   </joint>
-    <xacro:JM1 name="JM" prefix="L1" instance="1"  parent="arm2_1" />
+    <link name="arm2_2" />
+  <joint name="arm23_joint" type="revolute">
+    <origin xyz="0 0 0" rpy="0 ${pi/2} 0"/>
+    <child link="arm2_2"/>
+    <parent link="arm2_1"/>
+     <limit lower="${-pi}" upper="${pi}" effort="${max_effort}"
+      velocity="${max_velocity}" />
+  </joint>
+    <xacro:JM1 name="JM" prefix="L1" instance="1"  parent="arm2_2" />
     <xacro:PcModule parent="L11_PCmodule" prefix="L12" instance="2" />
     <xacro:PcModule parent="1_L1_j2_link" prefix="L11" instance="1" />
     <xacro:JM2 name="JM1" prefix="L1" instance="2"  parent="L12_PCmodule" reflect="0" shift="0.035" shift2="1"/>
-<!--
--->
+    <xacro:SMHand parent="2_L1_w1_link" prefix="L1" reflect="1" instance="2"/>
 <!--
  <xacro:SMRadprobe parent="2_L1_w1_link" prefix="L1" reflect="0" instance="1" />
+-->
+<!--
+    ARM3 - parent {instance}_${prefix}_camera_link
+-->
+        <link name="arm3" />
+<joint name="arm3_joint" type="revolute">
+    <origin xyz="0 0 0" rpy="0 ${pi/2} 0"/>
+    <child link="arm3"/>
+    <parent link="1_base_camera_link"/>
+     <limit lower="${-pi}" upper="${pi}" effort="${max_effort}"
+      velocity="${max_velocity}" />
+  </joint>
+  <link name="arm3_1" />
+  <joint name="arm32_joint" type="revolute">
+    <origin xyz="0 0 0" rpy="0 0 ${pi/2}"/>
+    <child link="arm3_1"/>
+    <parent link="arm3"/>
+     <limit lower="${-pi}" upper="${pi}" effort="${max_effort}"
+      velocity="${max_velocity}" />
+  </joint>
+    <link name="arm3_2" />
+  <joint name="arm33_joint" type="revolute">
+    <origin xyz="0 0 0" rpy="0 ${pi/2} 0"/>
+    <child link="arm3_2"/>
+    <parent link="arm3_1"/>
+     <limit lower="${-pi}" upper="${pi}" effort="${max_effort}"
+      velocity="${max_velocity}" />
+  </joint>
+    <xacro:JM1 name="JM" prefix="L3" instance="1"  parent="arm3_2" />
+    <xacro:PcModule parent="L31_PCmodule" prefix="L32" instance="2" />
+    <xacro:PcModule parent="1_L3_j2_link" prefix="L31" instance="1" />
+    <xacro:JM2 name="JM1" prefix="L3" instance="2"  parent="L32_PCmodule" reflect="0" shift="0.035" shift2="1"/>
+     <xacro:SMRadprobe parent="2_L3_w1_link" prefix="L3" reflect="0" instance="1" />
+<!--
+    <xacro:SMHand parent="2_L3_w1_link" prefix="L3" reflect="1" instance="3"/>
 -->
   <gazebo>

File: mrs_description/urdf/JM/jm.xacro (robot description, xacro)
@@ -7,4 +7,62 @@
   <!-- Import Rviz colors -->
   <xacro:include filename="$(find mrs_description)/urdf/materials.urdf.xacro" />
+<macro name="JM1_armconnect" params="name prefix instance parent">
+  <!-- Links -->
+  <create_link name="j1_link" color="Blue" mesh="${j1_mesh}"
+    cog="${j1_cog}" mass="${j1_mass}" instance="${instance}" prefix="${prefix}">
+    <j1_inertia />
+  </create_link>
+  <create_link_no_collision name="j2_link" color="Blue" mesh="${j2_mesh}"
+    cog="${j2_cog}" mass="${j2_mass}" instance="${instance}" prefix="${prefix}">
+    <j2_inertia />
+  </create_link_no_collision>
+  <create_link_no_collision name="j3_link" color="Blue" mesh="${j3_mesh}"
+    cog="${j3_cog}" mass="${j3_mass}" instance="${instance}" prefix="${prefix}">
+    <j3_inertia />
+  </create_link_no_collision>
+  <create_link name="w1_link" color="Blue" mesh="${w1_mesh}"
+    cog="${w1_cog}" mass="${w1_mass}" instance="${instance}" prefix="${prefix}">
+    <w1_inertia />
+  </create_link>
+  <!-- Joints -->
+  <joint name="${instance}_${prefix}_j3" type="continuous">
+    <child link="${instance}_${prefix}_w1_link" />
+    <parent link="${parent}" />
+    <axis xyz="0 0 1 " />
+    <origin xyz="0 0 0.01" rpy="${-pi/2} 0 0" />
+    <limit lower="${-pi/2}" upper="${pi/2}" effort="${max_effort}"
+      velocity="${max_velocity}" />
+    <dynamics damping="${j3_damping}" />
+ </joint>
+  <joint name="${instance}_${prefix}_j2_fixed" type="fixed">
+    <child link="${instance}_${prefix}_j3_link" />
+    <parent link="${instance}_${prefix}_w1_link" />
+    <origin xyz="0.045 0 0" rpy="0 0 ${pi/2}" />
+  </joint>
+  <joint name="${instance}_${prefix}_j2" type="revolute">
+    <child link="${instance}_${prefix}_j1_link" />
+    <parent link="${instance}_${prefix}_j3_link" />
+    <axis xyz="1 0 0 " />
+    <origin xyz="0 0 0" rpy="0 ${-pi/2} 0" />
+    <limit lower="${-pi/2}" upper="${pi/2}" effort="${max_effort}"
+      velocity="${max_velocity}" />
+    <dynamics damping="${j2_damping}" />
+  </joint>
+  <joint name="${instance}_${prefix}_j1" type="continuous">
+    <child link="${instance}_${prefix}_j2_link" />
+    <parent link="${instance}_${prefix}_j1_link" />
+    <axis xyz="0 0 1 " />
+    <origin xyz="0 -0.058 0" rpy="${pi/2} 0 0" />
+    <limit lower="${-pi/2}" upper="${pi/2}" effort="${max_effort}"
+      velocity="${max_velocity}" />
+    <dynamics damping="${j3_damping}" />
+  </joint>
+    <!-- Transmissions -->
+  <simple_transmission joint="${instance}_${prefix}_j1" />
+  <simple_transmission joint="${instance}_${prefix}_j2" />
+  <simple_transmission joint="${instance}_${prefix}_j3" />
+    <!-- Gazebo  -->
+  <xacro:JMG name="${name}_gazebo" prefix="${prefix}" instance="${instance}" />
+  </macro>
 <macro name="JM1" params="name prefix instance parent">
   <!-- Links -->
@@ -26,14 +84,20 @@
   </create_link>
   <!-- Joints -->
-  <joint name="${instance}_${prefix}_j3" type="fixed">
+<!--
+  <joint name="${instance}_${prefix}_j3" type="revolute">
     <child link="${instance}_${prefix}_w1_link" />
     <parent link="${parent}" />
     <axis xyz="0 0 1 " />
     <origin xyz="0 0 0.01" rpy="0 ${-pi/2} 0" />
-<!--
-    <limit lower="${-pi/2}" upper="${pi/2}" effort="${max_effort}"
-      velocity="${max_velocity}" />
-    <dynamics damping="${j3_damping}" />
--->
+    <limit lower="${-pi/2}" upper="${pi/2}" effort="${max_effort}"
+      velocity="${max_velocity}" />
+    <dynamics damping="${j3_damping}" />
+ </joint>
+-->
+    <joint name="${instance}_${prefix}_j3" type="fixed">
+    <child link="${instance}_${prefix}_w1_link" />
+    <parent link="${parent}" />
+    <axis xyz="0 0 1 " />
+    <origin xyz="0 0 0.01" rpy="0 ${-pi/2} 0" />
   </joint>
   <joint name="${instance}_${prefix}_j2_fixed" type="fixed">
@@ -334,5 +398,5 @@
   <xacro:JMG name="${name}_gazebo" prefix="${prefix}" instance="${instance}" />
   </macro>
-<macro name="JM3_solid" params="name prefix instance parent reflect shift">
+<macro name="JM3" params="name prefix instance parent reflect shift">
   <create_link name="j1_link" color="Blue" mesh="${j1_mesh}"
     cog="${j1_cog}" mass="${j1_mass}" instance="${instance}" prefix="${prefix}">
@@ -351,5 +415,5 @@
     <w1_inertia />
   </create_link>
-  <joint name="${instance}_${prefix}_j3" type="fixed">
+  <joint name="${instance}_${prefix}_j3" type="continuous">
     <child link="${instance}_${prefix}_w1_link" />
     <parent link="${instance}_${prefix}_j3_link" />
@@ -357,4 +421,57 @@
     <origin xyz="0 0.05 0" rpy="0 0 ${-pi/2}" />
   </joint>
+  <joint name="${instance}_${prefix}_j2" type="revolute">
+    <child link="${instance}_${prefix}_j3_link" />
+    <parent link="${instance}_${prefix}_j1_link" />
+    <axis xyz="0 0 1 " />
+    <origin xyz="0 0 0" rpy="0 ${pi/2} 0" />
+    <limit lower="${-pi/2}" upper="${pi/2}" effort="${max_effort}"
+      velocity="${max_velocity}" />
+    <dynamics damping="${j2_damping}" />
+  </joint>
+  <joint name="${instance}_${prefix}_j2_fixed" type="fixed">
+    <child link="${instance}_${prefix}_j1_link" />
+    <parent link="${instance}_${prefix}_j2_link" />
+    <axis xyz="1 0 0 " />
+    <origin xyz="0 0 0.058" rpy="${pi/2} 0 ${pi/2}" />
+  </joint>
+  <joint name="${instance}_${prefix}_j1" type="continuous">
+    <child link="${instance}_${prefix}_j2_link" />
+    <parent link="${parent}" />
+<!--
+    <axis xyz="1 0 0 " />
+-->
+    <origin xyz="${shift} 0 0" rpy="0 ${pi/2} 0" />
+  </joint>
+    <!-- Transmissions -->
+  <simple_transmission joint="${instance}_${prefix}_j1" />
+  <simple_transmission joint="${instance}_${prefix}_j2" />
+  <simple_transmission joint="${instance}_${prefix}_j3" />
+  <!-- Gazebo  -->
+  <xacro:JMG name="${name}_gazebo" prefix="${prefix}" instance="${instance}" />
+  </macro>
+<macro name="JM3_solid" params="name prefix instance parent reflect shift">
+  <create_link name="j1_link" color="Blue" mesh="${j1_mesh}"
+    cog="${j1_cog}" mass="${j1_mass}" instance="${instance}" prefix="${prefix}">
+    <j1_inertia />
+  </create_link>
+  <create_link_no_collision name="j2_link" color="Blue" mesh="${j2_mesh}"
+    cog="${j2_cog}" mass="${j2_mass}" instance="${instance}" prefix="${prefix}">
+    <j2_inertia />
+  </create_link_no_collision>
+  <create_link_no_collision name="j3_link" color="Blue" mesh="${j3_mesh}"
+    cog="${j3_cog}" mass="${j3_mass}" instance="${instance}" prefix="${prefix}">
+    <j3_inertia />
+  </create_link_no_collision>
+  <create_link name="w1_link" color="Blue" mesh="${w1_mesh}"
+    cog="${w1_cog}" mass="${w1_mass}" instance="${instance}" prefix="${prefix}">
+    <w1_inertia />
+  </create_link>
+  <joint name="${instance}_${prefix}_j3" type="fixed">
+    <child link="${instance}_${prefix}_w1_link" />
+    <parent link="${instance}_${prefix}_j3_link" />
+    <axis xyz="1 0 0" />
+    <origin xyz="0 0.05 0" rpy="0 0 ${-pi/2}" />
+  </joint>
   <joint name="${instance}_${prefix}_j2" type="fixed">
     <child link="${instance}_${prefix}_j3_link" />

File: mrs_description/urdf/power_base/base.urdf.xacro (robot description, xacro)
@@ -1,15 +1,9 @@
 <?xml version="1.0"?>
 <robot xmlns:xacro="http://www.ros.org/wiki/xacro">
-<xacro:include filename="$(find mrs_description)/urdf/power_base/ball_bearing.urdf.xacro" />
-    <!-- constants for robot -->
-<xacro:include filename="$(find mrs_description)/urdf/common_mrs.xacro" />
-  <!-- simplified box collision geometry for base -->
-<xacro:include filename="$(find
-mrs_description)/urdf/power_base/sm_other.urdf.xacro" />
   <property name="mass" value="22.0"/>
   <property name="p_baselen" value=".3" />
   <property name="p_basewidth" value=".3" />
-  <property name="p_baseheight" value=".6" />
-  <xacro:macro name="power_base" params="name">
+  <property name="p_baseheight" value=".3" />
+  <xacro:macro name="power_base" params="name parent">
   <link name="${name}_footprint">
     <inertial>
@@ -19,5 +13,5 @@
     </inertial>
     <visual>
-      <origin xyz="0 0 0" rpy="0 0 0"/>
+      <origin xyz="-2.2 0 0" rpy="0 0 0"/>
       <geometry>
         <box size="0.001 0.001 0.001"/>
@@ -32,4 +26,9 @@
     </collision>
   </link>
+  <joint name="${name}_footprint" type="fixed">
+    <origin xyz="0 0 0" rpy="0 0 0"/>
+    <child link="${name}_footprint"/>
+    <parent link="${parent}"/>
+  </joint>
   <joint name="${name}_footprint_joint" type="fixed">
     <origin xyz="0 0 0" rpy="0 0 0"/>
@@ -78,18 +77,20 @@
       </geometry>
     </collision>
-    <xacro:default_inertial mass="2" />
+    <xacro:default_inertial mass="2" I_tensor="1"/>
   </link>
   <gazebo reference="${name}_link_support">
     <material>Gazebo/Orange</material>
   </gazebo>
-<xacro:Ball_bearing mass="0.1" instance="1" dia="0.05" x="0.05" y="0.05" z="-0.29" parent="${name}_link_support"/>
-<xacro:Ball_bearing mass="0.1" instance="2" dia="0.05" x="-0.05" y="0.05" z="-0.29" parent="${name}_link_support"/>
-<xacro:Ball_bearing mass="0.1" instance="3" dia="0.05" x="0.05" y="-0.05" z="-0.29" parent="${name}_link_support"/>
-<xacro:Ball_bearing mass="0.1" instance="4" dia="0.05" x="-0.05" y="-0.05" z="-0.29" parent="${name}_link_support"/>
-<xacro:Camera parent="${name}_link_support" prefix="base" x="0.15" y="0" z="0.27" instance="1" />
-<xacro:Camera parent="${name}_link_support" prefix="base" x="0" y="0.15" z="0.27" instance="2" />
-<xacro:Camera parent="${name}_link_support" prefix="base" x="-0.15" y="0" z="0.27" instance="3" />
-<xacro:Camera parent="${name}_link_support" prefix="base" x="0" y="-0.15" z="0.27" instance="4" />
+<xacro:Ball_bearing mass="0.1" instance="1" dia="0.1" x="0.075" y="0.075" z="-0.12" parent="${name}_link_support"/>
+<xacro:Ball_bearing mass="0.1" instance="2" dia="0.1" x="-0.075" y="0.075" z="-0.12" parent="${name}_link_support"/>
+<xacro:Ball_bearing mass="0.1" instance="3" dia="0.1" x="0.075" y="-0.075" z="-0.12" parent="${name}_link_support"/>
+<xacro:Ball_bearing mass="0.1" instance="4" dia="0.1" x="-0.075" y="-0.075" z="-0.12" parent="${name}_link_support"/>
+<xacro:Camera parent="${name}_link_support" prefix="base" x="0.15" y="0" z="0.15" instance="1" />
+<xacro:Camera parent="${name}_link_support" prefix="base" x="0" y="0.15" z="0.15" instance="2" />
+<xacro:Camera parent="${name}_link_support" prefix="base" x="-0.15" y="0" z="0.15" instance="3" />
+<xacro:Camera parent="${name}_link_support" prefix="base" x="0" y="-0.15" z="0.15" instance="4" />
+<!--
 <xacro:Laser parent="${name}_link_support" prefix="base" x="0" y="0" z="0.31" instance="1" />
+-->
 <xacro:IMU parent="${name}_link_support" prefix="base" x="0.1" y="0.1" z="0.31"  />
   </xacro:macro>
